File: DuinoModSingle.sch (KiCad schematic (older format))
At the start: 12 parts, among them P1 CONN_02X03, U1 ATMEGA32U4-A, X1 16MHz

Commit message: schematic closer to complete
Parts:
- added C2, C4: 0.1uF, Capacitors_SMD:c_1206, symbol C
- added L1: Ferrite Bead, Capacitors_SMD:c_0805, symbol INDUCTOR_SMALL
- F1: footprint (none) -> Capacitors_SMD:c_1812; Manufacturer (none) -> Bourns; Part Number (none) -> MF-MSMF050-2
- VR1, VR2: Manufacturer (none) -> Bourns; Part Number (none) -> CG0603MLC-05E
- X1: Manufacturer (none) -> AVX; Part Number (none) -> PBRC16.00HR70X000
Connections:
- net +5V: now also U1.14 (VCC), U1.2 (UVCC), U1.34 (VCC), U1.44 (AVCC), C2.1, L1.1
- net GND: now also C2.2, C4.2
- net at U1.24 (AVCC): now also C4.1, L1.2
Changed lines of the file:
@@
 EESchema Schematic File Version 2
+LIBS:ReflowToaster
 LIBS:power
-LIBS:device_fixed
 LIBS:device
 LIBS:transistors
@@
 L +5V #PWR?
 U 1 1 540E8743
-P 5900 1750
-F 0 "#PWR?" H 5900 1840 20  0001 C CNN
-F 1 "+5V" H 5900 1840 30  0000 C CNN
-F 2 "" H 5900 1750 60  0000 C CNN
-F 3 "" H 5900 1750 60  0000 C CNN
-	1    5900 1750
-	1    0    0    -1
-$EndComp
-$Comp
-L +5V #PWR?
-U 1 1 540E875B
-P 5800 1750
-F 0 "#PWR?" H 5800 1840 20  0001 C CNN
-F 1 "+5V" H 5800 1840 30  0000 C CNN
-F 2 "" H 5800 1750 60  0000 C CNN
-F 3 "" H 5800 1750 60  0000 C CNN
-	1    5800 1750
+P 5900 1350
+F 0 "#PWR?" H 5900 1440 20  0001 C CNN
+F 1 "+5V" H 5900 1440 30  0000 C CNN
+F 2 "" H 5900 1350 60  0000 C CNN
+F 3 "" H 5900 1350 60  0000 C CNN
+	1    5900 1350
 	1    0    0    -1
 $EndComp
@@
 L +5V #PWR?
 U 1 1 540E8773
-P 5550 1750
-F 0 "#PWR?" H 5550 1840 20  0001 C CNN
-F 1 "+5V" H 5550 1840 30  0000 C CNN
-F 2 "" H 5550 1750 60  0000 C CNN
-F 3 "" H 5550 1750 60  0000 C CNN
-	1    5550 1750
+P 5550 1350
+F 0 "#PWR?" H 5550 1440 20  0001 C CNN
+F 1 "+5V" H 5550 1440 30  0000 C CNN
+F 2 "" H 5550 1350 60  0000 C CNN
+F 3 "" H 5550 1350 60  0000 C CNN
+	1    5550 1350
 	1    0    0    -1
 $EndComp
@@
 L +5V #PWR?
 U 1 1 540E878B
-P 5450 1750
-F 0 "#PWR?" H 5450 1840 20  0001 C CNN
-F 1 "+5V" H 5450 1840 30  0000 C CNN
-F 2 "" H 5450 1750 60  0000 C CNN
-F 3 "" H 5450 1750 60  0000 C CNN
-	1    5450 1750
+P 5450 1350
+F 0 "#PWR?" H 5450 1440 20  0001 C CNN
+F 1 "+5V" H 5450 1440 30  0000 C CNN
+F 2 "" H 5450 1350 60  0000 C CNN
+F 3 "" H 5450 1350 60  0000 C CNN
+	1    5450 1350
 	1    0    0    -1
 $EndComp
@@
 L +5V #PWR?
 U 1 1 540E87A3
-P 5200 1750
-F 0 "#PWR?" H 5200 1840 20  0001 C CNN
-F 1 "+5V" H 5200 1840 30  0000 C CNN
-F 2 "" H 5200 1750 60  0000 C CNN
-F 3 "" H 5200 1750 60  0000 C CNN
-	1    5200 1750
+P 5200 1350
+F 0 "#PWR?" H 5200 1440 20  0001 C CNN
+F 1 "+5V" H 5200 1440 30  0000 C CNN
+F 2 "" H 5200 1350 60  0000 C CNN
+F 3 "" H 5200 1350 60  0000 C CNN
+	1    5200 1350
 	1    0    0    -1
 $EndComp
@@
 F 1 "VR" V 3780 4160 40  0001 L CNN
 F 2 "Capacitors_SMD:c_0603" H 3780 4160 60  0001 C CNN
-F 3 "" H 3780 4160 60  0000 C CNN
+F 3 "http://datasheet.octopart.com/CG0603MLC-05E-Bourns-datasheet-17172219.pdf" H 3780 4160 60  0001 C CNN
+F 4 "Bourns" V 3750 4050 60  0001 C CNN "Manufacturer"
+F 5 "CG0603MLC-05E" V 3750 4050 60  0001 C CNN "Part Number"
 	1    3750 4050
 	1    0    0    -1
@@
 F 1 "VR" V 3630 4160 40  0001 L CNN
 F 2 "Capacitors_SMD:c_0603" H 3630 4160 60  0001 C CNN
-F 3 "" H 3630 4160 60  0000 C CNN
+F 3 "http://datasheet.octopart.com/CG0603MLC-05E-Bourns-datasheet-17172219.pdf" H 3630 4160 60  0001 C CNN
+F 4 "Bourns" V 3600 4050 60  0001 C CNN "Manufacturer"
+F 5 "CG0603MLC-05E" V 3600 4050 60  0001 C CNN "Part Number"
 	1    3600 4050
 	1    0    0    -1
@@
 F 0 "F1" H 3900 3550 40  0000 C CNN
 F 1 "500mA" H 3700 3450 40  0000 C CNN
-F 2 "" H 3800 3500 60  0000 C CNN
-F 3 "" H 3800 3500 60  0000 C CNN
+F 2 "Capacitors_SMD:c_1812" H 3800 3500 60  0001 C CNN
+F 3 " 	http://datasheet.octopart.com/MF-MSMF050-2-Bourns-datasheet-28511.pdf" H 3800 3500 60  0001 C CNN
+F 4 "Bourns" H 3800 3500 60  0001 C CNN "Manufacturer"
+F 5 "MF-MSMF050-2" H 3800 3500 60  0001 C CNN "Part Number"
 	1    3800 3500
 	1    0    0    -1
@@
 F 1 "16MHz" V 4600 2550 60  0000 C CNN
 F 2 "" H 4300 2800 60  0000 C CNN
-F 3 "" H 4300 2800 60  0000 C CNN
+F 3 "http://datasheet.octopart.com/PBRC16.00HR70X000-AVX-datasheet-2504.pdf" H 4300 2800 60  0001 C CNN
+F 4 "AVX" V 4300 2800 60  0001 C CNN "Manufacturer"
+F 5 "PBRC16.00HR70X000 " V 4300 2800 60  0001 C CNN "Part Number"
 	1    4300 2800
 	0    1    1    0
@@
 Wire Wire Line
 	3950 2800 4000 2800
+$Comp
+L INDUCTOR_SMALL L1
+U 1 1 540F28C4
+P 6300 1450
+F 0 "L1" H 6300 1550 50  0000 C CNN
+F 1 "Ferrite Bead" H 6300 1400 50  0001 C CNN
+F 2 "Capacitors_SMD:c_0805" H 6300 1450 60  0001 C CNN
+F 3 "http://www.bourns.com/data/global/pdfs/mh.pdf" H 6300 1450 60  0001 C CNN
+F 4 "Bourns" H 6300 1450 60  0001 C CNN "Manufacturer"
+F 5 "MH2029-300Y" H 6300 1450 60  0001 C CNN "Part Number"
+	1    6300 1450
+	1    0    0    -1
+$EndComp
+$Comp
+L C C4
+U 1 1 540F2AB3
+P 6650 1650
+F 0 "C4" H 6650 1750 40  0000 L CNN
+F 1 "0.1uF" H 6656 1565 40  0000 L CNN
+F 2 "Capacitors_SMD:c_1206" H 6688 1500 30  0001 C CNN
+F 3 "" H 6650 1650 60  0000 C CNN
+	1    6650 1650
+	1    0    0    -1
+$EndComp
+Wire Wire Line
+	5900 2050 5900 1350
+Wire Wire Line
+	5900 1450 6050 1450
+Connection ~ 5900 1450
+Wire Wire Line
+	6550 1450 6650 1450
+$Comp
+L GND #PWR?
+U 1 1 540F2D6C
+P 6650 1950
+F 0 "#PWR?" H 6650 1950 30  0001 C CNN
+F 1 "GND" H 6650 1880 30  0001 C CNN
+F 2 "" H 6650 1950 60  0000 C CNN
+F 3 "" H 6650 1950 60  0000 C CNN
+	1    6650 1950
+	1    0    0    -1
+$EndComp
+Wire Wire Line
+	6650 1950 6650 1850
+Wire Wire Line
+	6600 1450 6600 1550
+Wire Wire Line
+	6600 1550 5800 1550
+Wire Wire Line
+	5800 1550 5800 2050
+Connection ~ 6600 1450
+$Comp
+L C C2
+U 1 1 540F2F1E
+P 5650 1650
+F 0 "C2" H 5650 1750 40  0000 L CNN
+F 1 "0.1uF" H 5656 1565 40  0000 L CNN
+F 2 "Capacitors_SMD:c_1206" H 5688 1500 30  0001 C CNN
+F 3 "" H 5650 1650 60  0000 C CNN
+	1    5650 1650
+	1    0    0    -1
+$EndComp
+$Comp
+L GND #PWR?
+U 1 1 540F3001
+P 5650 1950
+F 0 "#PWR?" H 5650 1950 30  0001 C CNN
+F 1 "GND" H 5650 1880 30  0001 C CNN
+F 2 "" H 5650 1950 60  0000 C CNN
+F 3 "" H 5650 1950 60  0000 C CNN
+	1    5650 1950
+	1    0    0    -1
+$EndComp
+Wire Wire Line
+	5650 1950 5650 1850
+Wire Wire Line
+	5550 2050 5550 1350
+Wire Wire Line
+	5550 1450 5650 1450
+Connection ~ 5550 1450
+Wire Wire Line
+	5450 2050 5450 1350
+Wire Wire Line
+	5200 1350 5200 2050
 $EndSCHEMATC

Commit message: add footprint for resonator
Parts:
- U1: footprint TQFP44 -> SMD_Packages:TQFP-44
- X1: footprint (none) -> ReflowToaster:AVX_PBRC-H
Changed lines of the file:
@@
 F 0 "U1" H 4700 5550 40  0000 C CNN
 F 1 "ATMEGA32U4-A" H 6350 2350 40  0000 C CNN
-F 2 "TQFP44" H 5650 3850 35  0001 C CIN
+F 2 "SMD_Packages:TQFP-44" H 5650 3850 35  0001 C CIN
 F 3 "" H 6750 4950 60  0000 C CNN
 	1    5650 3850
@@
 	6750 4400 6800 4400
 $Comp
-L GND #PWR?
+L GND #PWR01
 U 1 1 540E7BE1
 P 7300 4450
-F 0 "#PWR?" H 7300 4450 30  0001 C CNN
+F 0 "#PWR01" H 7300 4450 30  0001 C CNN
 F 1 "GND" H 7300 4380 30  0001 C CNN
 F 2 "" H 7300 4450 60  0000 C CNN
@@
 Connection ~ 6950 2500
 $Comp
-L GND #PWR?
+L GND #PWR02
 U 1 1 540E8213
 P 8350 2600
-F 0 "#PWR?" H 8350 2600 30  0001 C CNN
+F 0 "#PWR02" H 8350 2600 30  0001 C CNN
 F 1 "GND" H 8350 2530 30  0001 C CNN
 F 2 "" H 8350 2600 60  0000 C CNN
@@
 	8350 2550 8300 2550
 $Comp
-L +5V #PWR?
+L +5V #PWR03
 U 1 1 540E8258
 P 8350 2050
-F 0 "#PWR?" H 8350 2140 20  0001 C CNN
+F 0 "#PWR03" H 8350 2140 20  0001 C CNN
 F 1 "+5V" H 8350 2140 30  0000 C CNN
 F 2 "" H 8350 2050 60  0000 C CNN
@@
 	4450 2300 4500 2300
 $Comp
-L +5V #PWR?
+L +5V #PWR04
 U 1 1 540E8743
 P 5900 1350
-F 0 "#PWR?" H 5900 1440 20  0001 C CNN
+F 0 "#PWR04" H 5900 1440 20  0001 C CNN
 F 1 "+5V" H 5900 1440 30  0000 C CNN
 F 2 "" H 5900 1350 60  0000 C CNN
@@
 $EndComp
 $Comp
-L +5V #PWR?
+L +5V #PWR05
 U 1 1 540E8773
 P 5550 1350
-F 0 "#PWR?" H 5550 1440 20  0001 C CNN
+F 0 "#PWR05" H 5550 1440 20  0001 C CNN
 F 1 "+5V" H 5550 1440 30  0000 C CNN
 F 2 "" H 5550 1350 60  0000 C CNN
@@
 $EndComp
 $Comp
-L +5V #PWR?
+L +5V #PWR06
 U 1 1 540E878B
 P 5450 1350
-F 0 "#PWR?" H 5450 1440 20  0001 C CNN
+F 0 "#PWR06" H 5450 1440 20  0001 C CNN
 F 1 "+5V" H 5450 1440 30  0000 C CNN
 F 2 "" H 5450 1350 60  0000 C CNN
@@
 $EndComp
 $Comp
-L +5V #PWR?
+L +5V #PWR07
 U 1 1 540E87A3
 P 5200 1350
-F 0 "#PWR?" H 5200 1440 20  0001 C CNN
+F 0 "#PWR07" H 5200 1440 20  0001 C CNN
 F 1 "+5V" H 5200 1440 30  0000 C CNN
 F 2 "" H 5200 1350 60  0000 C CNN
@@
 $EndComp
 $Comp
-L GND #PWR?
+L GND #PWR08
 U 1 1 540E87C7
 P 5800 5500
-F 0 "#PWR?" H 5800 5500 30  0001 C CNN
+F 0 "#PWR08" H 5800 5500 30  0001 C CNN
 F 1 "GND" H 5800 5430 30  0001 C CNN
 F 2 "" H 5800 5500 60  0000 C CNN
@@
 $EndComp
 $Comp
-L GND #PWR?
+L GND #PWR09
 U 1 1 540E87DF
 P 5700 5500
-F 0 "#PWR?" H 5700 5500 30  0001 C CNN
+F 0 "#PWR09" H 5700 5500 30  0001 C CNN
 F 1 "GND" H 5700 5430 30  0001 C CNN
 F 2 "" H 5700 5500 60  0000 C CNN
@@
 $EndComp
 $Comp
-L GND #PWR?
+L GND #PWR010
 U 1 1 540E87F7
 P 5600 5500
-F 0 "#PWR?" H 5600 5500 30  0001 C CNN
+F 0 "#PWR010" H 5600 5500 30  0001 C CNN
 F 1 "GND" H 5600 5430 30  0001 C CNN
 F 2 "" H 5600 5500 60  0000 C CNN
@@
 $EndComp
 $Comp
-L GND #PWR?
+L GND #PWR011
 U 1 1 540E880F
 P 5500 5500
-F 0 "#PWR?" H 5500 5500 30  0001 C CNN
+F 0 "#PWR011" H 5500 5500 30  0001 C CNN
 F 1 "GND" H 5500 5430 30  0001 C CNN
 F 2 "" H 5500 5500 60  0000 C CNN
@@
 $EndComp
 $Comp
-L GND #PWR?
+L GND #PWR012
 U 1 1 540E883E
 P 5250 5500
-F 0 "#PWR?" H 5250 5500 30  0001 C CNN
+F 0 "#PWR012" H 5250 5500 30  0001 C CNN
 F 1 "GND" H 5250 5430 30  0001 C CNN
 F 2 "" H 5250 5500 60  0000 C CNN
@@
 $EndComp
 $Comp
-L GND #PWR?
+L GND #PWR013
 U 1 1 540E8BE8
 P 4400 5200
-F 0 "#PWR?" H 4400 5200 30  0001 C CNN
+F 0 "#PWR013" H 4400 5200 30  0001 C CNN
 F 1 "GND" H 4400 5130 30  0001 C CNN
 F 2 "" H 4400 5200 60  0000 C CNN
@@
 $EndComp
 $Comp
-L GND #PWR?
+L GND #PWR014
 U 1 1 540E8E03
 P 4400 4400
-F 0 "#PWR?" H 4400 4400 30  0001 C CNN
+F 0 "#PWR014" H 4400 4400 30  0001 C CNN
 F 1 "GND" H 4400 4330 30  0001 C CNN
 F 2 "" H 4400 4400 60  0000 C CNN
@@
 Connection ~ 3750 3650
 $Comp
-L GND #PWR?
+L GND #PWR015
 U 1 1 540E90E0
 P 3750 4350
-F 0 "#PWR?" H 3750 4350 30  0001 C CNN
+F 0 "#PWR015" H 3750 4350 30  0001 C CNN
 F 1 "GND" H 3750 4280 30  0001 C CNN
 F 2 "" H 3750 4350 60  0000 C CNN
@@
 $EndComp
 $Comp
-L GND #PWR?
+L GND #PWR016
 U 1 1 540E90FE
 P 3600 4350
-F 0 "#PWR?" H 3600 4350 30  0001 C CNN
+F 0 "#PWR016" H 3600 4350 30  0001 C CNN
 F 1 "GND" H 3600 4280 30  0001 C CNN
 F 2 "" H 3600 4350 60  0000 C CNN
@@
 	4050 3500 4500 3500
 $Comp
-L +5V #PWR?
+L +5V #PWR017
 U 1 1 540E9337
 P 4450 3450
-F 0 "#PWR?" H 4450 3540 20  0001 C CNN
+F 0 "#PWR017" H 4450 3540 20  0001 C CNN
 F 1 "+5V" H 4450 3540 30  0000 C CNN
 F 2 "" H 4450 3450 60  0000 C CNN
@@
 F 0 "X1" V 4150 2900 60  0000 C CNN
 F 1 "16MHz" V 4600 2550 60  0000 C CNN
-F 2 "" H 4300 2800 60  0000 C CNN
+F 2 "ReflowToaster:AVX_PBRC-H" H 4300 2800 60  0001 C CNN
 F 3 "http://datasheet.octopart.com/PBRC16.00HR70X000-AVX-datasheet-2504.pdf" H 4300 2800 60  0001 C CNN
 F 4 "AVX" V 4300 2800 60  0001 C CNN "Manufacturer"
@@
 	4500 3100 4500 2900
 $Comp
-L GND #PWR?
+L GND #PWR018
 U 1 1 540E91B1
 P 3950 2850
-F 0 "#PWR?" H 3950 2850 30  0001 C CNN
+F 0 "#PWR018" H 3950 2850 30  0001 C CNN
 F 1 "GND" H 3950 2780 30  0001 C CNN
 F 2 "" H 3950 2850 60  0000 C CNN
@@
 	6550 1450 6650 1450
 $Comp
-L GND #PWR?
+L GND #PWR019
 U 1 1 540F2D6C
 P 6650 1950
-F 0 "#PWR?" H 6650 1950 30  0001 C CNN
+F 0 "#PWR019" H 6650 1950 30  0001 C CNN
 F 1 "GND" H 6650 1880 30  0001 C CNN
 F 2 "" H 6650 1950 60  0000 C CNN
@@
 $EndComp
 $Comp
-L GND #PWR?
+L GND #PWR020
 U 1 1 540F3001
 P 5650 1950
-F 0 "#PWR?" H 5650 1950 30  0001 C CNN
+F 0 "#PWR020" H 5650 1950 30  0001 C CNN
 F 1 "GND" H 5650 1880 30  0001 C CNN
 F 2 "" H 5650 1950 60  0000 C CNN

Commit message: DuinoModSingle complete
Parts:
- added C5, C6: 1uF, Capacitors_SMD:c_1206, symbol C
- added U2: MCP1700T-3302E/TT, SMD_Packages:SOT-23, symbol MCP1700T-3302E/TT
Connections:
- net +5V: now also C6.1, U2.3 (Vin)
- net GND: now also C5.2, C6.2, U2.1 (GND)
- new net +3.3V: C5.1, U2.2 (Vout)
Other:
- moved on the sheet: C1, C2, C3, C4, F1, L1, P1, R1, R2, R3, R4, U1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

Commit message: more changes
Changed lines of the file:
@@
 EESchema Schematic File Version 2
+LIBS:transistors
 LIBS:ReflowToaster
+LIBS:device
+LIBS:conn
 LIBS:power
-LIBS:device
-LIBS:transistors
-LIBS:conn
-LIBS:linear
-LIBS:regul
-LIBS:74xx
-LIBS:cmos4000
-LIBS:adc-dac
-LIBS:memory
-LIBS:xilinx
-LIBS:special
-LIBS:microcontrollers
-LIBS:dsp
-LIBS:microchip
-LIBS:analog_switches
-LIBS:motorola
-LIBS:texas
-LIBS:intel
-LIBS:audio
-LIBS:interface
-LIBS:digital-audio
-LIBS:philips
-LIBS:display
-LIBS:cypress
-LIBS:siliconi
-LIBS:opto
-LIBS:atmel
-LIBS:contrib
-LIBS:valves
 LIBS:ReflowToaster-cache
 EELAYER 24 0
@@
 Text HLabel 1800 4550 3    60   Output ~ 0
 +5V
-Text HLabel 1950 4400 1    60   Output ~ 0
+Text HLabel 1950 4400 1    60   UnSpc ~ 0
 GND
 Wire Wire Line
