File: DuinoModSingle.sch (KiCad schematic (older format))
At the start: 18 parts, among them P1 CONN_02X03, U1 ATMEGA32U4-A, U2 MCP1700T-3302E/TT, X1 16MHz

Commit message: DuinoModSingle & main sheet tagged with vendor part #s for BOM generation
Parts:
- C1, C5, C6: DigiKey P/N (none) -> 399-8147-1-ND; Manufacturer (none) -> Kemet; Mouser P/N (none) -> 80-C1206C105K5R; Part Number (none) -> C1206C105K5RACTU
- C2, C3, C4: DigiKey P/N (none) -> 399-1249-1-ND; Manufacturer (none) -> Kemet; Mouser P/N (none) -> 80-C1206C104K5R; Part Number (none) -> C1206C104K5RACTU
- F1': renamed from F1; DigiKey P/N (none) -> MF-MSMF050-2CT-ND; Mouser P/N (none) -> 652-MF-MSMF050-2
- L1: DigiKey P/N (none) -> MH2029-300YCT-ND; Mouser P/N (none) -> 652-MH2029-300Y
- P1: DigiKey P/N (none) -> 952-2120-ND; Manufacturer (none) -> Harwin; Mouser P/N (none) -> 855-M20-9980345; Part Number (none) -> M20-9980345
- R1, R2: DigiKey P/N (none) -> P22ECT-ND; Manufacturer (none) -> Panasonic; Mouser P/N (none) -> 667-ERJ-8GEYJ220V; Part Number (none) -> ERJ-8GEYJ220V
- R3, R4: DigiKey P/N (none) -> P10KECT-ND; Manufacturer (none) -> Panasonic; Mouser P/N (none) -> 667-ERJ-8GEYJ103V; Part Number (none) -> ERJ-8GEYJ103V
- U1: DigiKey P/N (none) -> ATMEGA32U4-AURCT-ND; Manufacturer (none) -> Atmel; Mouser P/N (none) -> 556-ATMEGA32U4-AU; Part Number (none) -> ATMEGA32U4-AU
- U2: DigiKey P/N (none) -> MCP1700T3302ETTCT-ND; Mouser P/N (none) -> 579-MCP1700T3302E/TT
- VR1, VR2: DigiKey P/N (none) -> CG0603MLC-05ECT-ND; Mouser P/N (none) -> 652-CG0603MLC-05E
- X1: DigiKey P/N (none) -> 1253-1084-1-ND; Mouser P/N (none) -> 581-PBRC1600HR70X000
Changed lines of the file:
@@
 F 1 "ATMEGA32U4-A" H 6400 3100 40  0000 C CNN
 F 2 "SMD_Packages:TQFP-44" H 5700 4600 35  0001 C CIN
-F 3 "" H 6800 5700 60  0000 C CNN
+F 3 "http://www.atmel.com/Images/Atmel-7766-8-bit-AVR-ATmega16U4-32U4_%20Datasheet.pdf" H 6800 5700 60  0001 C CNN
+F 4 "Atmel" H 3500 3550 60  0001 C CNN "Manufacturer"
+F 5 "ATMEGA32U4-AU" H 3500 3550 60  0001 C CNN "Part Number"
+F 6 "ATMEGA32U4-AURCT-ND" H 0   0   50  0001 C CNN "DigiKey P/N"
+F 7 "556-ATMEGA32U4-AU" H 0   0   50  0001 C CNN "Mouser P/N"
 	1    5700 4600
 	1    0    0    -1
@@
 F 1 "10k" V 7132 5261 40  0000 L CNN
 F 2 "Capacitors_SMD:c_1206" V 7030 5150 30  0001 C CNN
-F 3 "" H 7125 5260 30  0000 C CNN
+F 3 "http://industrial.panasonic.com/www-cgi/jvcr13pz.cgi?E+PZ+3+AOA0001+ERJ8GEYJ103V+7+WW" H 7125 5260 30  0001 C CNN
+F 4 "Panasonic" H 3500 3550 60  0001 C CNN "Manufacturer"
+F 5 "ERJ-8GEYJ103V" H 3500 3550 60  0001 C CNN "Part Number"
+F 6 "P10KECT-ND" H 0   0   50  0001 C CNN "DigiKey P/N"
+F 7 "667-ERJ-8GEYJ103V" H 0   0   50  0001 C CNN "Mouser P/N"
 	1    7100 5150
 	0    1    1    0
@@
 F 1 "CONN_02X03" H 8100 3000 50  0001 C CNN
 F 2 "Socket_Strips:Socket_Strip_Straight_2x03" H 8100 2000 60  0001 C CNN
-F 3 "" H 8100 2000 60  0000 C CNN
+F 3 "http://harwin.com/includes/pdfs/M20-998.pdf" H 7125 5260 30  0001 C CNN
+F 4 "Harwin" H 3500 3550 60  0001 C CNN "Manufacturer"
+F 5 "M20-9980345" H 3500 3550 60  0001 C CNN "Part Number"
+F 6 "952-2120-ND" H 0   0   50  0001 C CNN "DigiKey P/N"
+F 7 "855-M20-9980345" H 0   0   50  0001 C CNN "Mouser P/N"
 	1    8100 3200
 	1    0    0    -1
@@
 F 1 "10k" V 8132 2961 40  0000 L CNN
 F 2 "Capacitors_SMD:c_1206" V 8030 2850 30  0001 C CNN
-F 3 "" H 8125 2960 30  0000 C CNN
+F 3 "http://industrial.panasonic.com/www-cgi/jvcr13pz.cgi?E+PZ+3+AOA0001+ERJ8GEYJ103V+7+WW" H 7125 5260 30  0001 C CNN
+F 4 "Panasonic" H 3500 3550 60  0001 C CNN "Manufacturer"
+F 5 "ERJ-8GEYJ103V" H 3500 3550 60  0001 C CNN "Part Number"
+F 6 "P10KECT-ND" H 0   0   50  0001 C CNN "DigiKey P/N"
+F 7 "667-ERJ-8GEYJ103V" H 0   0   50  0001 C CNN "Mouser P/N"
 	1    8100 2850
 	0    1    1    0
@@
 F 1 "0.1uF" H 4456 5615 40  0000 L CNN
 F 2 "Capacitors_SMD:c_1206" H 4488 5550 30  0001 C CNN
-F 3 "" H 4450 5700 60  0000 C CNN
+F 3 "http://www.kemet.com/docfinder?Partnumber=C1206C104K5RACTU" H 7125 5260 30  0001 C CNN
+F 4 "Kemet" H 3500 3550 60  0001 C CNN "Manufacturer"
+F 5 "C1206C104K5RACTU" H 3500 3550 60  0001 C CNN "Part Number"
+F 6 "399-1249-1-ND" H 0   0   50  0001 C CNN "DigiKey P/N"
+F 7 "80-C1206C104K5R" H 0   0   50  0001 C CNN "Mouser P/N"
 	1    4450 5700
 	1    0    0    -1
@@
 F 1 "1uF" H 4456 4815 40  0000 L CNN
 F 2 "Capacitors_SMD:c_1206" H 4488 4750 30  0001 C CNN
-F 3 "" H 4450 4900 60  0000 C CNN
+F 3 "http://www.kemet.com/docfinder?Partnumber=C1206C105K5RACTU" H 7125 5260 30  0001 C CNN
+F 4 "Kemet" H 3500 3550 60  0001 C CNN "Manufacturer"
+F 5 "C1206C105K5RACTU" H 3500 3550 60  0001 C CNN "Part Number"
+F 6 "399-8147-1-ND" H 0   0   50  0001 C CNN "DigiKey P/N"
+F 7 "80-C1206C105K5R" H 0   0   50  0001 C CNN "Mouser P/N"
 	1    4450 4900
 	1    0    0    -1
@@
 F 1 "22" V 4232 4511 40  0000 L CNN
 F 2 "Capacitors_SMD:c_1206" H 4130 4400 30  0001 C CNN
-F 3 "" H 4225 4510 30  0000 C CNN
+F 3 "http://industrial.panasonic.com/www-cgi/jvcr13pz.cgi?E+PZ+3+AOA0001+ERJ8GEYJ220V+7+WW" H 7125 5260 30  0001 C CNN
+F 4 "Panasonic" H 3500 3550 60  0001 C CNN "Manufacturer"
+F 5 "ERJ-8GEYJ220V" H 3500 3550 60  0001 C CNN "Part Number"
+F 6 "P22ECT-ND" H 0   0   50  0001 C CNN "DigiKey P/N"
+F 7 "667-ERJ-8GEYJ220V" H 0   0   50  0001 C CNN "Mouser P/N"
 	1    4200 4400
 	0    1    1    0
@@
 F 1 "22" V 4132 4611 40  0000 L CNN
 F 2 "Capacitors_SMD:c_1206" H 4030 4500 30  0001 C CNN
-F 3 "" H 4125 4610 30  0000 C CNN
+F 3 "http://industrial.panasonic.com/www-cgi/jvcr13pz.cgi?E+PZ+3+AOA0001+ERJ8GEYJ220V+7+WW" H 7125 5260 30  0001 C CNN
+F 4 "Panasonic" H 3500 3550 60  0001 C CNN "Manufacturer"
+F 5 "ERJ-8GEYJ220V" H 3500 3550 60  0001 C CNN "Part Number"
+F 6 "P22ECT-ND" H 0   0   50  0001 C CNN "DigiKey P/N"
+F 7 "667-ERJ-8GEYJ220V" H 0   0   50  0001 C CNN "Mouser P/N"
 	1    4100 4500
 	0    1    1    0
@@
 F 1 "VR" V 3830 4910 40  0001 L CNN
 F 2 "Capacitors_SMD:c_0603" H 3830 4910 60  0001 C CNN
-F 3 "http://datasheet.octopart.com/CG0603MLC-05E-Bourns-datasheet-17172219.pdf" H 3830 4910 60  0001 C CNN
+F 3 "http://www.bourns.com/data/global/pdfs/MLC.pdf" H 3830 4910 60  0001 C CNN
 F 4 "Bourns" V 3800 4800 60  0001 C CNN "Manufacturer"
 F 5 "CG0603MLC-05E" V 3800 4800 60  0001 C CNN "Part Number"
+F 6 "CG0603MLC-05ECT-ND" H 0   0   50  0001 C CNN "DigiKey P/N"
+F 7 "652-CG0603MLC-05E" H 0   0   50  0001 C CNN "Mouser P/N"
 	1    3800 4800
 	1    0    0    -1
@@
 F 1 "VR" V 3680 4910 40  0001 L CNN
 F 2 "Capacitors_SMD:c_0603" H 3680 4910 60  0001 C CNN
-F 3 "http://datasheet.octopart.com/CG0603MLC-05E-Bourns-datasheet-17172219.pdf" H 3680 4910 60  0001 C CNN
-F 4 "Bourns" V 3650 4800 60  0001 C CNN "Manufacturer"
-F 5 "CG0603MLC-05E" V 3650 4800 60  0001 C CNN "Part Number"
+F 3 "http://www.bourns.com/data/global/pdfs/MLC.pdf" H 3830 4910 60  0001 C CNN
+F 4 "Bourns" V 3800 4800 60  0001 C CNN "Manufacturer"
+F 5 "CG0603MLC-05E" V 3800 4800 60  0001 C CNN "Part Number"
+F 6 "CG0603MLC-05ECT-ND" H 0   0   50  0001 C CNN "DigiKey P/N"
+F 7 "652-CG0603MLC-05E" H 0   0   50  0001 C CNN "Mouser P/N"
 	1    3650 4800
 	1    0    0    -1
@@
 	3800 5050 3800 5100
 $Comp
-L FUSE F1
+L FUSE F1'
 U 1 1 540E91CF
 P 3850 4250
@@
 F 1 "500mA" H 3750 4200 40  0000 C CNN
 F 2 "Capacitors_SMD:c_1812" H 3850 4250 60  0001 C CNN
-F 3 " 	http://datasheet.octopart.com/MF-MSMF050-2-Bourns-datasheet-28511.pdf" H 3850 4250 60  0001 C CNN
+F 3 "http://www.bourns.com/data/global/pdfs/mfmsmf.pdf" H 3850 4250 60  0001 C CNN
 F 4 "Bourns" H 3850 4250 60  0001 C CNN "Manufacturer"
 F 5 "MF-MSMF050-2" H 3850 4250 60  0001 C CNN "Part Number"
+F 6 "MF-MSMF050-2CT-ND" H 0   0   50  0001 C CNN "DigiKey P/N"
+F 7 "652-MF-MSMF050-2" H 0   0   50  0001 C CNN "Mouser P/N"
 	1    3850 4250
 	1    0    0    -1
@@
 F 1 "16MHz" V 4650 3300 60  0000 C CNN
 F 2 "ReflowToaster:AVX_PBRC-H" H 4350 3550 60  0001 C CNN
-F 3 "http://datasheet.octopart.com/PBRC16.00HR70X000-AVX-datasheet-2504.pdf" H 4350 3550 60  0001 C CNN
+F 3 "http://global.kyocera.com/prdct/electro/pdf/resonator/pbr-ce.pdf" H 4350 3550 60  0001 C CNN
 F 4 "AVX" V 4350 3550 60  0001 C CNN "Manufacturer"
 F 5 "PBRC16.00HR70X000 " V 4350 3550 60  0001 C CNN "Part Number"
+F 6 "1253-1084-1-ND" H 0   0   50  0001 C CNN "DigiKey P/N"
+F 7 "581-PBRC1600HR70X000" H 0   0   50  0001 C CNN "Mouser P/N"
 	1    4350 3550
 	0    1    1    0
@@
 F 4 "Bourns" H 6350 2200 60  0001 C CNN "Manufacturer"
 F 5 "MH2029-300Y" H 6350 2200 60  0001 C CNN "Part Number"
+F 6 "MH2029-300YCT-ND" H 0   0   50  0001 C CNN "DigiKey P/N"
+F 7 "652-MH2029-300Y" H 0   0   50  0001 C CNN "Mouser P/N"
 	1    6350 2200
 	1    0    0    -1
@@
 F 1 "0.1uF" H 6706 2315 40  0000 L CNN
 F 2 "Capacitors_SMD:c_1206" H 6738 2250 30  0001 C CNN
-F 3 "" H 6700 2400 60  0000 C CNN
+F 3 "http://www.kemet.com/docfinder?Partnumber=C1206C104K5RACTU" H 7125 5260 30  0001 C CNN
+F 4 "Kemet" H 3500 3550 60  0001 C CNN "Manufacturer"
+F 5 "C1206C104K5RACTU" H 3500 3550 60  0001 C CNN "Part Number"
+F 6 "399-1249-1-ND" H 0   0   50  0001 C CNN "DigiKey P/N"
+F 7 "80-C1206C104K5R" H 0   0   50  0001 C CNN "Mouser P/N"
 	1    6700 2400
 	1    0    0    -1
@@
 F 1 "0.1uF" H 5706 2315 40  0000 L CNN
 F 2 "Capacitors_SMD:c_1206" H 5738 2250 30  0001 C CNN
-F 3 "" H 5700 2400 60  0000 C CNN
+F 3 "http://www.kemet.com/docfinder?Partnumber=C1206C104K5RACTU" H 7125 5260 30  0001 C CNN
+F 4 "Kemet" H 3500 3550 60  0001 C CNN "Manufacturer"
+F 5 "C1206C104K5RACTU" H 3500 3550 60  0001 C CNN "Part Number"
+F 6 "399-1249-1-ND" H 0   0   50  0001 C CNN "DigiKey P/N"
+F 7 "80-C1206C104K5R" H 0   0   50  0001 C CNN "Mouser P/N"
 	1    5700 2400
 	1    0    0    -1
@@
 F 4 "Microchip" H 2150 2550 60  0001 C CNN "Manufacturer"
 F 5 "MCP1700T-3302E/TT" H 2675 2625 60  0001 C CNN "Part Number"
+F 6 "MCP1700T3302ETTCT-ND" H 0   0   50  0001 C CNN "DigiKey P/N"
+F 7 "579-MCP1700T3302E/TT" H 0   0   50  0001 C CNN "Mouser P/N"
 	1    2000 3150
 	1    0    0    -1
@@
 F 1 "1uF" H 1556 3315 40  0000 L CNN
 F 2 "Capacitors_SMD:c_1206" H 1588 3250 30  0001 C CNN
-F 3 "" H 1550 3400 60  0000 C CNN
+F 3 "http://www.kemet.com/docfinder?Partnumber=C1206C105K5RACTU" H 7125 5260 30  0001 C CNN
+F 4 "Kemet" H 3500 3550 60  0001 C CNN "Manufacturer"
+F 5 "C1206C105K5RACTU" H 3500 3550 60  0001 C CNN "Part Number"
+F 6 "399-8147-1-ND" H 0   0   50  0001 C CNN "DigiKey P/N"
+F 7 "80-C1206C105K5R" H 0   0   50  0001 C CNN "Mouser P/N"
 	1    1550 3400
 	1    0    0    -1
@@
 F 1 "1uF" H 2456 3315 40  0000 L CNN
 F 2 "Capacitors_SMD:c_1206" H 2488 3250 30  0001 C CNN
-F 3 "" H 2450 3400 60  0000 C CNN
+F 3 "http://www.kemet.com/docfinder?Partnumber=C1206C105K5RACTU" H 7125 5260 30  0001 C CNN
+F 4 "Kemet" H 3500 3550 60  0001 C CNN "Manufacturer"
+F 5 "C1206C105K5RACTU" H 3500 3550 60  0001 C CNN "Part Number"
+F 6 "399-8147-1-ND" H 0   0   50  0001 C CNN "DigiKey P/N"
+F 7 "80-C1206C105K5R" H 0   0   50  0001 C CNN "Mouser P/N"
 	1    2450 3400
 	1    0    0    -1

Commit message: remove some extra whitespace
Parts:
- X1: Part Number PBRC16.00HR70X000 -> PBRC16.00HR70X000
Changed lines of the file:
@@
 F 3 "http://global.kyocera.com/prdct/electro/pdf/resonator/pbr-ce.pdf" H 4350 3550 60  0001 C CNN
 F 4 "AVX" V 4350 3550 60  0001 C CNN "Manufacturer"
-F 5 "PBRC16.00HR70X000 " V 4350 3550 60  0001 C CNN "Part Number"
+F 5 "PBRC16.00HR70X000" V 4350 3550 60  0001 C CNN "Part Number"
 F 6 "1253-1084-1-ND" H 0   0   50  0001 C CNN "DigiKey P/N"
 F 7 "581-PBRC1600HR70X000" H 0   0   50  0001 C CNN "Mouser P/N"

Commit message: last of the new footprints added; PCB started
Parts:
- renumbered F1' to F1
Changed lines of the file:
@@
 	3800 5050 3800 5100
 $Comp
-L FUSE F1'
+L FUSE F1
 U 1 1 540E91CF
 P 3850 4250

Commit message: redo annotation
Parts:
- renumbered C6 to C1, C5 to C2, C1 to C3, C3 to C4, C2 to C5, C4 to C6, R4 to R3, R3 to R4, U2 to U1, U1 to U2
Changed lines of the file:
@@
 $EndDescr
 $Comp
-L ATMEGA32U4-A U1
+L ATMEGA32U4-A U2
 U 1 1 540E78F9
 P 5700 4600
-F 0 "U1" H 4750 6300 40  0000 C CNN
+F 0 "U2" H 4750 6300 40  0000 C CNN
 F 1 "ATMEGA32U4-A" H 6400 3100 40  0000 C CNN
 F 2 "SMD_Packages:TQFP-44" H 5700 4600 35  0001 C CIN
@@
 	6900 5750 6800 5750
 $Comp
-L R R4
+L R R3
 U 1 1 540E7B32
 P 7100 5150
-F 0 "R4" V 7065 5055 40  0000 R CNN
+F 0 "R3" V 7065 5055 40  0000 R CNN
 F 1 "10k" V 7132 5261 40  0000 L CNN
 F 2 "Capacitors_SMD:c_1206" V 7030 5150 30  0001 C CNN
@@
 	6800 5150 6850 5150
 $Comp
-L GND #PWR013
+L GND #PWR38
 U 1 1 540E7BE1
 P 7350 5200
-F 0 "#PWR013" H 7350 5200 30  0001 C CNN
+F 0 "#PWR38" H 7350 5200 30  0001 C CNN
 F 1 "GND" H 7350 5130 30  0001 C CNN
 F 2 "" H 7350 5200 60  0000 C CNN
@@
 Connection ~ 7000 3250
 $Comp
-L GND #PWR014
+L GND #PWR40
 U 1 1 540E8213
 P 8400 3350
-F 0 "#PWR014" H 8400 3350 30  0001 C CNN
+F 0 "#PWR40" H 8400 3350 30  0001 C CNN
 F 1 "GND" H 8400 3280 30  0001 C CNN
 F 2 "" H 8400 3350 60  0000 C CNN
@@
 	8400 3300 8350 3300
 $Comp
-L +5V #PWR015
+L +5V #PWR39
 U 1 1 540E8258
 P 8400 2800
-F 0 "#PWR015" H 8400 2890 20  0001 C CNN
+F 0 "#PWR39" H 8400 2890 20  0001 C CNN
 F 1 "+5V" H 8400 2890 30  0000 C CNN
 F 2 "" H 8400 2800 60  0000 C CNN
@@
 	6800 3750 7050 3750
 $Comp
-L R R3
+L R R4
 U 1 1 540E83F6
 P 8100 2850
-F 0 "R3" V 8065 2755 40  0000 R CNN
+F 0 "R4" V 8065 2755 40  0000 R CNN
 F 1 "10k" V 8132 2961 40  0000 L CNN
 F 2 "Capacitors_SMD:c_1206" V 8030 2850 30  0001 C CNN
@@
 	4500 3050 4550 3050
 $Comp
-L +5V #PWR016
+L +5V #PWR36
 U 1 1 540E8743
 P 5950 2100
-F 0 "#PWR016" H 5950 2190 20  0001 C CNN
+F 0 "#PWR36" H 5950 2190 20  0001 C CNN
 F 1 "+5V" H 5950 2190 30  0000 C CNN
 F 2 "" H 5950 2100 60  0000 C CNN
@@
 $EndComp
 $Comp
-L +5V #PWR017
+L +5V #PWR31
 U 1 1 540E8773
 P 5600 2100
-F 0 "#PWR017" H 5600 2190 20  0001 C CNN
+F 0 "#PWR31" H 5600 2190 20  0001 C CNN
 F 1 "+5V" H 5600 2190 30  0000 C CNN
 F 2 "" H 5600 2100 60  0000 C CNN
@@
 $EndComp
 $Comp
-L +5V #PWR018
+L +5V #PWR29
 U 1 1 540E878B
 P 5500 2100
-F 0 "#PWR018" H 5500 2190 20  0001 C CNN
+F 0 "#PWR29" H 5500 2190 20  0001 C CNN
 F 1 "+5V" H 5500 2190 30  0000 C CNN
 F 2 "" H 5500 2100 60  0000 C CNN
@@
 $EndComp
 $Comp
-L +5V #PWR019
+L +5V #PWR27
 U 1 1 540E87A3
 P 5250 2100
-F 0 "#PWR019" H 5250 2190 20  0001 C CNN
+F 0 "#PWR27" H 5250 2190 20  0001 C CNN
 F 1 "+5V" H 5250 2190 30  0000 C CNN
 F 2 "" H 5250 2100 60  0000 C CNN
@@
 $EndComp
 $Comp
-L GND #PWR020
+L GND #PWR35
 U 1 1 540E87C7
 P 5850 6250
-F 0 "#PWR020" H 5850 6250 30  0001 C CNN
+F 0 "#PWR35" H 5850 6250 30  0001 C CNN
 F 1 "GND" H 5850 6180 30  0001 C CNN
 F 2 "" H 5850 6250 60  0000 C CNN
@@
 $EndComp
 $Comp
-L GND #PWR021
+L GND #PWR34
 U 1 1 540E87DF
 P 5750 6250
-F 0 "#PWR021" H 5750 6250 30  0001 C CNN
+F 0 "#PWR34" H 5750 6250 30  0001 C CNN
 F 1 "GND" H 5750 6180 30  0001 C CNN
 F 2 "" H 5750 6250 60  0000 C CNN
@@
 $EndComp
 $Comp
-L GND #PWR022
+L GND #PWR32
 U 1 1 540E87F7
 P 5650 6250
-F 0 "#PWR022" H 5650 6250 30  0001 C CNN
+F 0 "#PWR32" H 5650 6250 30  0001 C CNN
 F 1 "GND" H 5650 6180 30  0001 C CNN
 F 2 "" H 5650 6250 60  0000 C CNN
@@
 $EndComp
 $Comp
-L GND #PWR023
+L GND #PWR30
 U 1 1 540E880F
 P 5550 6250
-F 0 "#PWR023" H 5550 6250 30  0001 C CNN
+F 0 "#PWR30" H 5550 6250 30  0001 C CNN
 F 1 "GND" H 5550 6180 30  0001 C CNN
 F 2 "" H 5550 6250 60  0000 C CNN
@@
 $EndComp
 $Comp
-L GND #PWR024
+L GND #PWR28
 U 1 1 540E883E
 P 5300 6250
-F 0 "#PWR024" H 5300 6250 30  0001 C CNN
+F 0 "#PWR28" H 5300 6250 30  0001 C CNN
 F 1 "GND" H 5300 6180 30  0001 C CNN
 F 2 "" H 5300 6250 60  0000 C CNN
@@
 	5850 6250 5850 6200
 $Comp
-L C C3
+L C C4
 U 1 1 540E8B06
 P 4450 5700
-F 0 "C3" H 4450 5800 40  0000 L CNN
+F 0 "C4" H 4450 5800 40  0000 L CNN
 F 1 "0.1uF" H 4456 5615 40  0000 L CNN
 F 2 "Capacitors_SMD:c_1206" H 4488 5550 30  0001 C CNN
@@
 $EndComp
 $Comp
-L GND #PWR025
+L GND #PWR25
 U 1 1 540E8BE8
 P 4450 5950
-F 0 "#PWR025" H 4450 5950 30  0001 C CNN
+F 0 "#PWR25" H 4450 5950 30  0001 C CNN
 F 1 "GND" H 4450 5880 30  0001 C CNN
 F 2 "" H 4450 5950 60  0000 C CNN
@@
 Connection ~ 4450 5450
 $Comp
-L C C1
+L C C3
 U 1 1 540E8D92
 P 4450 4900
-F 0 "C1" H 4450 5000 40  0000 L CNN
+F 0 "C3" H 4450 5000 40  0000 L CNN
 F 1 "1uF" H 4456 4815 40  0000 L CNN
 F 2 "Capacitors_SMD:c_1206" H 4488 4750 30  0001 C CNN
@@
 $EndComp
 $Comp
-L GND #PWR026
+L GND #PWR24
 U 1 1 540E8E03
 P 4450 5150
-F 0 "#PWR026" H 4450 5150 30  0001 C CNN
+F 0 "#PWR24" H 4450 5150 30  0001 C CNN
 F 1 "GND" H 4450 5080 30  0001 C CNN
 F 2 "" H 4450 5150 60  0000 C CNN
@@
 Connection ~ 3800 4400
 $Comp
-L GND #PWR027
+L GND #PWR22
 U 1 1 540E90E0
 P 3800 5100
-F 0 "#PWR027" H 3800 5100 30  0001 C CNN
+F 0 "#PWR22" H 3800 5100 30  0001 C CNN
 F 1 "GND" H 3800 5030 30  0001 C CNN
 F 2 "" H 3800 5100 60  0000 C CNN
@@
 $EndComp
 $Comp
-L GND #PWR028
+L GND #PWR21
 U 1 1 540E90FE
 P 3650 5100
-F 0 "#PWR028" H 3650 5100 30  0001 C CNN
+F 0 "#PWR21" H 3650 5100 30  0001 C CNN
 F 1 "GND" H 3650 5030 30  0001 C CNN
 F 2 "" H 3650 5100 60  0000 C CNN
@@
 	4100 4250 4550 4250
 $Comp
-L +5V #PWR029
+L +5V #PWR26
 U 1 1 540E9337
 P 4500 4200
-F 0 "#PWR029" H 4500 4290 20  0001 C CNN
+F 0 "#PWR26" H 4500 4290 20  0001 C CNN
 F 1 "+5V" H 4500 4290 30  0000 C CNN
 F 2 "" H 4500 4200 60  0000 C CNN
@@
 	4550 3850 4550 3650
 $Comp
-L GND #PWR030
+L GND #PWR23
 U 1 1 540E91B1
 P 4000 3600
-F 0 "#PWR030" H 4000 3600 30  0001 C CNN
+F 0 "#PWR23" H 4000 3600 30  0001 C CNN
 F 1 "GND" H 4000 3530 30  0001 C CNN
 F 2 "" H 4000 3600 60  0000 C CNN
@@
 $EndComp
 $Comp
-L C C4
+L C C6
 U 1 1 540F2AB3
 P 6700 2400
-F 0 "C4" H 6700 2500 40  0000 L CNN
+F 0 "C6" H 6700 2500 40  0000 L CNN
 F 1 "0.1uF" H 6706 2315 40  0000 L CNN
 F 2 "Capacitors_SMD:c_1206" H 6738 2250 30  0001 C CNN
@@
 	6600 2200 6700 2200
 $Comp
-L GND #PWR031
+L GND #PWR37
 U 1 1 540F2D6C
 P 6700 2700
-F 0 "#PWR031" H 6700 2700 30  0001 C CNN
+F 0 "#PWR37" H 6700 2700 30  0001 C CNN
 F 1 "GND" H 6700 2630 30  0001 C CNN
 F 2 "" H 6700 2700 60  0000 C CNN
@@
 Connection ~ 6650 2200
 $Comp
-L C C2
+L C C5
 U 1 1 540F2F1E
 P 5700 2400
-F 0 "C2" H 5700 2500 40  0000 L CNN
+F 0 "C5" H 5700 2500 40  0000 L CNN
 F 1 "0.1uF" H 5706 2315 40  0000 L CNN
 F 2 "Capacitors_SMD:c_1206" H 5738 2250 30  0001 C CNN
@@
 $EndComp
 $Comp
-L GND #PWR032
+L GND #PWR33
 U 1 1 540F3001
 P 5700 2700
-F 0 "#PWR032" H 5700 2700 30  0001 C CNN
+F 0 "#PWR33" H 5700 2700 30  0001 C CNN
 F 1 "GND" H 5700 2630 30  0001 C CNN
 F 2 "" H 5700 2700 60  0000 C CNN
@@
 	5250 2100 5250 2800
 $Comp
-L MCP1700T-3302E/TT U2
+L MCP1700T-3302E/TT U1
 U 1 1 540F663F
 P 2000 3150
-F 0 "U2" H 1700 3300 60  0000 L CNN
+F 0 "U1" H 1700 3300 60  0000 L CNN
 F 1 "MCP1700T-3302E/TT" H 1550 2500 60  0000 L CNN
 F 2 "SMD_Packages:SOT-23" H 1400 2600 60  0001 C CNN
@@
 $EndComp
 $Comp
-L C C6
+L C C1
 U 1 1 540F6784
 P 1550 3400
-F 0 "C6" H 1550 3500 40  0000 L CNN
+F 0 "C1" H 1550 3500 40  0000 L CNN
 F 1 "1uF" H 1556 3315 40  0000 L CNN
 F 2 "Capacitors_SMD:c_1206" H 1588 3250 30  0001 C CNN
@@
 $EndComp
 $Comp
-L C C5
+L C C2
 U 1 1 540F6815
 P 2450 3400
-F 0 "C5" H 2450 3500 40  0000 L CNN
+F 0 "C2" H 2450 3500 40  0000 L CNN
 F 1 "1uF" H 2456 3315 40  0000 L CNN
 F 2 "Capacitors_SMD:c_1206" H 2488 3250 30  0001 C CNN
@@
 $EndComp
 $Comp
-L GND #PWR033
+L GND #PWR20
 U 1 1 540F69EC
 P 2450 3650
-F 0 "#PWR033" H 2450 3650 30  0001 C CNN
+F 0 "#PWR20" H 2450 3650 30  0001 C CNN
 F 1 "GND" H 2450 3580 30  0001 C CNN
 F 2 "" H 2450 3650 60  0000 C CNN
@@
 $EndComp
 $Comp
-L GND #PWR034
+L GND #PWR14
 U 1 1 540F6A00
 P 1550 3650
-F 0 "#PWR034" H 1550 3650 30  0001 C CNN
+F 0 "#PWR14" H 1550 3650 30  0001 C CNN
 F 1 "GND" H 1550 3580 30  0001 C CNN
 F 2 "" H 1550 3650 60  0000 C CNN
@@
 $EndComp
 $Comp
-L GND #PWR035
+L GND #PWR18
 U 1 1 540F6A14
 P 2000 3650
-F 0 "#PWR035" H 2000 3650 30  0001 C CNN
+F 0 "#PWR18" H 2000 3650 30  0001 C CNN
 F 1 "GND" H 2000 3580 30  0001 C CNN
 F 2 "" H 2000 3650 60  0000 C CNN
@@
 $EndComp
 $Comp
-L +3.3V #PWR036
+L +3.3V #PWR19
 U 1 1 540F6A49
 P 2450 2900
-F 0 "#PWR036" H 2450 2860 30  0001 C CNN
+F 0 "#PWR19" H 2450 2860 30  0001 C CNN
 F 1 "+3.3V" H 2450 3010 30  0000 C CNN
 F 2 "" H 2450 2900 60  0000 C CNN
@@
 $EndComp
 $Comp
-L +5V #PWR037
+L +5V #PWR13
 U 1 1 540F6A5D
 P 1550 2900
-F 0 "#PWR037" H 1550 2990 20  0001 C CNN
+F 0 "#PWR13" H 1550 2990 20  0001 C CNN
 F 1 "+5V" H 1550 2990 30  0000 C CNN
 F 2 "" H 1550 2900 60  0000 C CNN
@@
 Connection ~ 2450 3150
 $Comp
-L +3.3V #PWR038
+L +3.3V #PWR15
 U 1 1 540F96E9
 P 1650 4450
-F 0 "#PWR038" H 1650 4410 30  0001 C CNN
+F 0 "#PWR15" H 1650 4410 30  0001 C CNN
 F 1 "+3.3V" H 1650 4560 30  0000 C CNN
 F 2 "" H 1650 4450 60  0000 C CNN
@@
 $EndComp
 $Comp
-L +5V #PWR039
+L +5V #PWR16
 U 1 1 540F9745
 P 1800 4450
-F 0 "#PWR039" H 1800 4540 20  0001 C CNN
+F 0 "#PWR16" H 1800 4540 20  0001 C CNN
 F 1 "+5V" H 1800 4540 30  0000 C CNN
 F 2 "" H 1800 4450 60  0000 C CNN
@@
 $EndComp
 $Comp
-L GND #PWR040
+L GND #PWR17
 U 1 1 540F9759
 P 1950 4500
-F 0 "#PWR040" H 1950 4500 30  0001 C CNN
+F 0 "#PWR17" H 1950 4500 30  0001 C CNN
 F 1 "GND" H 1950 4430 30  0001 C CNN
 F 2 "" H 1950 4500 60  0000 C CNN
