File: ReflowToaster.sch (KiCad schematic (older format))
At the start: 0 parts

Commit message: DuinoModSingle complete
Changed lines of the file:
@@
 Sheet 1 2
 Title "ReflowToaster"
-Date "08 Sep 2014"
-Rev ""
-Comp ""
+Date "09 September 2014"
+Rev "0.1"
+Comp "Scott Alfter"
 Comment1 ""
 Comment2 ""
@@
 $EndDescr
 $Sheet
-S 11200 0    1300 2800
+S 4700 1950 1100 2800
 U 540E7838
 F0 "DuinoModSingle" 60
 F1 "DuinoModSingle.sch" 60
+F2 "A5" B R 5800 2050 60
+F3 "A4" B R 5800 2150 60
+F4 "A3" B R 5800 2250 60
+F5 "A2" B R 5800 2350 60
+F6 "A1" B R 5800 2450 60
+F7 "A0" B R 5800 2550 60
+F8 "7" B R 5800 3600 60
+F9 "3/SCL/PWM" B R 5800 4000 60
+F10 "2/SDA" B R 5800 4100 60
+F11 "0/RX" B R 5800 4300 60
+F12 "1/TX" B R 5800 4200 60
+F13 "4/A6" B R 5800 3900 60
+F14 "12/A7" B R 5800 3100 60
+F15 "6/PWM/A8" B R 5800 3700 60
+F16 "5/PWM" B R 5800 3800 60
+F17 "13/PWM" B R 5800 3000 60
+F18 "SCK" B R 5800 4450 60
+F19 "MOSI" B R 5800 4550 60
+F20 "MISO" B R 5800 4650 60
+F21 "8/A9" B R 5800 3500 60
+F22 "9/PWM/A10" B R 5800 3400 60
+F23 "10/PWM/A11" B R 5800 3300 60
+F24 "11/PWM" B R 5800 3200 60
+F25 "~RESET" I L 4700 2350 60
+F26 "AREF" I L 4700 2550 60
+F27 "USB_D+" B L 4700 3600 60
+F28 "USB_D-" B L 4700 3500 60
+F29 "USB_5V" I L 4700 3700 60
+F30 "+3.3V" O L 4700 2150 60
+F31 "+5V" O L 4700 2050 60
+F32 "GND" O L 4700 4650 60
 $EndSheet
 $EndSCHEMATC

Commit message: more changes
Parts:
- added J2, J3: USB-Micro-B, symbol USB-Micro-B
- added Q1: FDN340P, SMD_Packages:SOT-23, symbol MOSFET_P
Connections:
- net DuinoModSingle/USB_5V: now also Q1.S
- net DuinoModSingle/USB_D+: now also J2.3 (D+)
- net DuinoModSingle/USB_D-: now also J2.2 (D-)
- new net: J2.1 (VBUS), Q1.D
- new net: J3.1 (VBUS), Q1.G
- new net GND: J2.10 (SHELL5), J2.11 (SHELL6), J2.4 (ID), J2.5 (GND), J2.6 (SHELL1), J2.7 (SHELL2), J2.8 (SHELL3), J2.9 (SHELL4), J3.10 (SHELL5), J3.11 (SHELL6), J3.4 (ID), J3.5 (GND), J3.6 (SHELL1), J3.7 (SHELL2), J3.8 (SHELL3), J3.9 (SHELL4)

Commit message: add footprint for USB connectors
Parts:
- J2, J3: footprint (none) -> ReflowToaster:FCI_10118192-0001LF
Changed lines of the file:
@@
 EESchema Schematic File Version 2
-LIBS:transistors
 LIBS:ReflowToaster
 LIBS:device
-LIBS:conn
+LIBS:atmel
 LIBS:power
 LIBS:ReflowToaster-cache
@@
 F 0 "J2" H 1350 4800 60  0000 C CNN
 F 1 "USB-Micro-B" H 1550 3850 60  0001 C CNN
-F 2 "" H 1600 4350 60  0000 C CNN
+F 2 "ReflowToaster:FCI_10118192-0001LF" H 1600 4350 60  0001 C CNN
 F 3 "http://www.mouser.com/ds/2/154/10118192AC-197249.pdf" H 1600 4350 60  0001 C CNN
 F 4 "FCI" H 1600 4350 60  0001 C CNN "Manufacturer"
@@
 F 0 "J3" H 1350 3750 60  0000 C CNN
 F 1 "USB-Micro-B" H 1550 2800 60  0001 C CNN
-F 2 "" H 1600 3300 60  0000 C CNN
+F 2 "ReflowToaster:FCI_10118192-0001LF" H 1600 3300 60  0001 C CNN
 F 3 "http://www.mouser.com/ds/2/154/10118192AC-197249.pdf" H 1600 3300 60  0001 C CNN
 F 4 "FCI" H 1600 3300 60  0001 C CNN "Manufacturer"

Commit message: add FDN340P
Parts:
- removed Q1: FDN340P, SMD_Packages:SOT-23, symbol MOSFET_P
- added Q1: FDN340P, ReflowToaster:FDN340P, symbol FDN340P
Connections:
- net DuinoModSingle/USB_5V: now also Q1.S
- net at J2.1 (VBUS): now also Q1.D
- net at J3.1 (VBUS): now also Q1.G
Changed lines of the file:
@@
 $EndSheet
-$Comp
-L MOSFET_P Q1
-U 1 1 540FD30D
-P 2500 3950
-F 0 "Q1" V 2400 4150 60  0000 R CNN
-F 1 "FDN340P" V 2700 4150 60  0000 R CNN
-F 2 "SMD_Packages:SOT-23" H 2500 3950 60  0001 C CNN
-F 3 "http://datasheet.octopart.com/FDN340P-Fairchild-datasheet-31668.pdf" H 2500 3950 60  0001 C CNN
-F 4 "Fairchild" H 2500 3950 60  0001 C CNN "Manufacturer"
-F 5 "FDN340P" H 2500 3950 60  0001 C CNN "Part Number"
-	1    2500 3950
-	0    -1   1    0
-$EndComp
 $Comp
 L USB-Micro-B J2
@@
 $EndComp
 $Comp
-L GND #PWR?
+L GND #PWR01
 U 1 1 540F85D9
 P 2200 4700
-F 0 "#PWR?" H 2200 4700 30  0001 C CNN
+F 0 "#PWR01" H 2200 4700 30  0001 C CNN
 F 1 "GND" H 2200 4630 30  0001 C CNN
 F 2 "" H 2200 4700 60  0000 C CNN
@@
 $EndComp
 $Comp
-L GND #PWR?
+L GND #PWR02
 U 1 1 540F86BE
 P 1000 4650
-F 0 "#PWR?" H 1000 4650 30  0001 C CNN
+F 0 "#PWR02" H 1000 4650 30  0001 C CNN
 F 1 "GND" H 1000 4580 30  0001 C CNN
 F 2 "" H 1000 4650 60  0000 C CNN
@@
 $EndComp
 $Comp
-L GND #PWR?
+L GND #PWR03
 U 1 1 540F9794
 P 2200 3650
-F 0 "#PWR?" H 2200 3650 30  0001 C CNN
+F 0 "#PWR03" H 2200 3650 30  0001 C CNN
 F 1 "GND" H 2200 3580 30  0001 C CNN
 F 2 "" H 2200 3650 60  0000 C CNN
@@
 $EndComp
 $Comp
-L GND #PWR?
+L GND #PWR04
 U 1 1 540F97A8
 P 1000 3600
-F 0 "#PWR?" H 1000 3600 30  0001 C CNN
+F 0 "#PWR04" H 1000 3600 30  0001 C CNN
 F 1 "GND" H 1000 3530 30  0001 C CNN
 F 2 "" H 1000 3600 60  0000 C CNN
@@
 $EndComp
 $Comp
-L GND #PWR?
+L GND #PWR05
 U 1 1 540F9DBA
 P 2700 5300
-F 0 "#PWR?" H 2700 5300 30  0001 C CNN
+F 0 "#PWR05" H 2700 5300 30  0001 C CNN
 F 1 "GND" H 2700 5230 30  0001 C CNN
 F 2 "" H 2700 5300 60  0000 C CNN
@@
 $EndComp
 $Comp
-L +5V #PWR?
+L +5V #PWR06
 U 1 1 540F9FAE
 P 2700 2700
-F 0 "#PWR?" H 2700 2790 20  0001 C CNN
+F 0 "#PWR06" H 2700 2790 20  0001 C CNN
 F 1 "+5V" H 2700 2790 30  0000 C CNN
 F 2 "" H 2700 2700 60  0000 C CNN
@@
 $EndComp
 $Comp
-L +3.3V #PWR?
+L +3.3V #PWR07
 U 1 1 540F9FC2
 P 2550 2700
-F 0 "#PWR?" H 2550 2660 30  0001 C CNN
+F 0 "#PWR07" H 2550 2660 30  0001 C CNN
 F 1 "+3.3V" H 2550 2810 30  0000 C CNN
 F 2 "" H 2550 2700 60  0000 C CNN
@@
 Wire Wire Line
 	2500 3650 2500 3750
+$Comp
+L FDN340P Q1
+U 1 1 540FC488
+P 2500 3950
+F 0 "Q1" V 2300 4100 60  0000 R CNN
+F 1 "FDN340P" V 2650 4150 60  0000 R CNN
+F 2 "ReflowToaster:FDN340P" H 2500 4900 60  0001 C CNN
+F 3 "http://datasheet.octopart.com/FDN340P-Fairchild-datasheet-31668.pdf" H 2500 5000 60  0001 C CNN
+F 4 "Fairchild" H 2500 5100 60  0001 C CNN "Manufacturer"
+F 5 "FDN340P" H 2500 5200 60  0001 C CNN "Part Number"
+	1    2500 3950
+	0    -1   1    0
+$EndComp
 $EndSCHEMATC
