File: Thermocouple.sch (KiCad schematic (older format))
At the start: 12 parts, among them J7 CONN_01X02, U5 74LVC2G34, U6 74LVC1T45, U7 MAX31855KASA+, U8 NUP2105L

Commit message: components tagged with vendor part IDs
Parts:
- C10, C11, C12, C9: DigiKey P/N (none) -> 399-1249-1-ND; Manufacturer (none) -> Kemet; Mouser P/N (none) -> 80-C1206C104K5R; Part Number (none) -> C1206C104K5RACTU
- C13: DigiKey P/N (none) -> 399-1234-1-ND; Manufacturer (none) -> Kemet; Mouser P/N (none) -> 80-C1206C103K5R; Part Number (none) -> C1206C103K5RACTU
- J7: DigiKey P/N (none) -> A98076-ND; Mouser P/N (none) -> 571-2828362
- L2, L3: DigiKey P/N (none) -> 490-1060-1-ND; Mouser P/N (none) -> 81-BLM41PG471SN1L
- U5: DigiKey P/N (none) -> 296-13496-1-ND; Mouser P/N (none) -> 595-SN74LVC2G34DBVR
- U6: DigiKey P/N (none) -> 296-16843-1-ND; Mouser P/N (none) -> 595-SN74LVC1T45DBVR
- U7: DigiKey P/N (none) -> MAX31855KASA+TCT-ND; Mouser P/N (none) -> 700-MAX31855KASA+
- U8: DigiKey P/N (none) -> NUP2105LT1GOSCT-ND; Mouser P/N (none) -> 863-NUP2105LT1G
Changed lines of the file:
@@
 F 4 "Maxim" H 5550 4975 60  0001 C CNN "Manufacturer"
 F 5 "MAX31855KASA+" H 5550 5050 60  0001 C CNN "Part Number"
+F 6 "MAX31855KASA+TCT-ND" H 0   0   50  0001 C CNN "DigiKey P/N"
+F 7 "700-MAX31855KASA+" H 0   0   50  0001 C CNN "Mouser P/N"
 	1    5550 3950
 	1    0    0    -1
@@
 F 1 "74LVC2G34" H 4650 3400 40  0000 C CNN
 F 2 "SMD_Packages:SOT-23-6" H 4650 3550 60  0001 C CNN
-F 3 "http://datasheet.octopart.com/SN74LVC2G34DBVR-Texas-Instruments-datasheet-153323.pdf" H 4650 3550 60  0001 C CNN
+F 3 "http://www.ti.com/lit/ds/symlink/sn74lvc2g34.pdf" H 4650 3550 60  0001 C CNN
 F 4 "Texas Instruments" H 4650 3550 60  0001 C CNN "Manufacturer"
 F 5 "SN74LVC2G34DBVR" H 4650 3550 60  0001 C CNN "Part Number"
+F 6 "296-13496-1-ND" H 0   0   50  0001 C CNN "DigiKey P/N"
+F 7 "595-SN74LVC2G34DBVR" H 0   0   50  0001 C CNN "Mouser P/N"
 	1    4650 3550
 	1    0    0    -1
@@
 F 1 "0.1uF" H 4656 4465 40  0000 L CNN
 F 2 "Capacitors_SMD:c_1206" H 4688 4400 30  0001 C CNN
-F 3 "" H 4650 4550 60  0000 C CNN
-F 4 "U5 Bypass" H 4850 4400 40  0000 C CNN "Usage"
+F 3 "http://www.kemet.com/docfinder?Partnumber=C1206C104K5RACTU" H 7125 5260 30  0001 C CNN
+F 4 "Kemet" H 3500 3550 60  0001 C CNN "Manufacturer"
+F 5 "C1206C104K5RACTU" H 3500 3550 60  0001 C CNN "Part Number"
+F 6 "399-1249-1-ND" H 0   0   50  0001 C CNN "DigiKey P/N"
+F 7 "80-C1206C104K5R" H 0   0   50  0001 C CNN "Mouser P/N"
+F 8 "U5 Bypass" H 4850 4400 40  0000 C CNN "Usage"
 	1    4650 4550
 	1    0    0    -1
@@
 F 1 "0.1uF" V 5800 3450 40  0000 L CNN
 F 2 "Capacitors_SMD:c_1206" H 5788 3250 30  0001 C CNN
-F 3 "" H 5750 3400 60  0000 C CNN
+F 3 "http://www.kemet.com/docfinder?Partnumber=C1206C104K5RACTU" H 7125 5260 30  0001 C CNN
+F 4 "Kemet" H 3500 3550 60  0001 C CNN "Manufacturer"
+F 5 "C1206C104K5RACTU" H 3500 3550 60  0001 C CNN "Part Number"
+F 6 "399-1249-1-ND" H 0   0   50  0001 C CNN "DigiKey P/N"
+F 7 "80-C1206C104K5R" H 0   0   50  0001 C CNN "Mouser P/N"
 	1    5750 3400
 	0    1    1    0
@@
 F 1 "74LVC1T45" H 3775 4650 60  0000 L CNN
 F 2 "SMD_Packages:SOT-23-6" H 3750 4950 60  0001 C CNN
-F 3 "http://datasheet.octopart.com/SN74LVC1T45DBVR-Texas-Instruments-datasheet-21259457.pdf" H 3750 5825 60  0001 C CNN
+F 3 "http://www.ti.com/lit/ds/symlink/sn74lvc1t45.pdf" H 3750 5825 60  0001 C CNN
 F 4 "Texas Instruments" H 3750 4950 60  0001 C CNN "Manufacturer"
 F 5 "SN74LVC1T45DBVR" H 3750 4950 60  0001 C CNN "Part Number"
+F 6 "296-16843-1-ND" H 0   0   50  0001 C CNN "DigiKey P/N"
+F 7 "595-SN74LVC1T45DBVR" H 0   0   50  0001 C CNN "Mouser P/N"
 	1    3750 4950
 	1    0    0    -1
@@
 F 1 "0.1uF" H 3556 4165 40  0000 L CNN
 F 2 "Capacitors_SMD:c_1206" H 3588 4100 30  0001 C CNN
-F 3 "" H 3550 4250 60  0000 C CNN
+F 3 "http://www.kemet.com/docfinder?Partnumber=C1206C104K5RACTU" H 7125 5260 30  0001 C CNN
+F 4 "Kemet" H 3500 3550 60  0001 C CNN "Manufacturer"
+F 5 "C1206C104K5RACTU" H 3500 3550 60  0001 C CNN "Part Number"
+F 6 "399-1249-1-ND" H 0   0   50  0001 C CNN "DigiKey P/N"
+F 7 "80-C1206C104K5R" H 0   0   50  0001 C CNN "Mouser P/N"
 	1    3550 4250
 	1    0    0    -1
@@
 F 1 "0.1uF" H 3956 4165 40  0000 L CNN
 F 2 "Capacitors_SMD:c_1206" H 3988 4100 30  0001 C CNN
-F 3 "" H 3950 4250 60  0000 C CNN
+F 3 "http://www.kemet.com/docfinder?Partnumber=C1206C104K5RACTU" H 7125 5260 30  0001 C CNN
+F 4 "Kemet" H 3500 3550 60  0001 C CNN "Manufacturer"
+F 5 "C1206C104K5RACTU" H 3500 3550 60  0001 C CNN "Part Number"
+F 6 "399-1249-1-ND" H 0   0   50  0001 C CNN "DigiKey P/N"
+F 7 "80-C1206C104K5R" H 0   0   50  0001 C CNN "Mouser P/N"
 	1    3950 4250
 	1    0    0    -1
@@
 F 1 "0.01uF" H 6456 3865 40  0000 L CNN
 F 2 "Capacitors_SMD:c_1206" H 6488 3800 30  0001 C CNN
-F 3 "" H 6450 3950 60  0000 C CNN
+F 3 "http://www.kemet.com/docfinder?Partnumber=C1206C103K5RACTU" H 7125 5260 30  0001 C CNN
+F 4 "Kemet" H 3500 3550 60  0001 C CNN "Manufacturer"
+F 5 "C1206C103K5RACTU" H 3500 3550 60  0001 C CNN "Part Number"
+F 6 "399-1234-1-ND" H 0   0   50  0001 C CNN "DigiKey P/N"
+F 7 "80-C1206C103K5R" H 0   0   50  0001 C CNN "Mouser P/N"
 	1    6450 3950
 	1    0    0    -1
@@
 F 4 "ON Semiconductor" H 6900 4450 60  0001 C CNN "Manufacturer"
 F 5 "NUP2105LT1G" H 6900 4450 60  0001 C CNN "Part Number"
+F 6 "NUP2105LT1GOSCT-ND" H 0   0   50  0001 C CNN "DigiKey P/N"
+F 7 "863-NUP2105LT1G" H 0   0   50  0001 C CNN "Mouser P/N"
 	1    6900 4450
 	1    0    0    -1
@@
 F 1 "INDUCTOR_SMALL" H 7400 3700 50  0001 C CNN
 F 2 "ReflowToaster:smd_1806" H 7400 3750 60  0001 C CNN
-F 3 "http://datasheet.octopart.com/BLM41PG471SN1L-Murata-datasheet-531466.pdf" H 7400 3750 60  0001 C CNN
+F 3 "http://search.murata.co.jp/Ceramy/image/img/PDF/ENG/L0110S0100BLM41P.pdf" H 7400 3750 60  0001 C CNN
 F 4 "Murata" H 7400 3750 60  0001 C CNN "Manufacturer"
 F 5 "BLM41PG471SN1L" H 7400 3750 60  0001 C CNN "Part Number"
+F 6 "490-1060-1-ND" H 0   0   50  0001 C CNN "DigiKey P/N"
+F 7 "81-BLM41PG471SN1L" H 0   0   50  0001 C CNN "Mouser P/N"
 	1    7400 3750
 	1    0    0    -1
@@
 F 1 "INDUCTOR_SMALL" H 7400 4100 50  0001 C CNN
 F 2 "ReflowToaster:smd_1806" H 7400 4150 60  0001 C CNN
-F 3 "http://datasheet.octopart.com/BLM41PG471SN1L-Murata-datasheet-531466.pdf" H 7400 4150 60  0001 C CNN
-F 4 "Murata" H 7400 4150 60  0001 C CNN "Manufacturer"
-F 5 "BLM41PG471SN1L" H 7400 4150 60  0001 C CNN "Part Number"
+F 3 "http://search.murata.co.jp/Ceramy/image/img/PDF/ENG/L0110S0100BLM41P.pdf" H 7400 3750 60  0001 C CNN
+F 4 "Murata" H 7400 3750 60  0001 C CNN "Manufacturer"
+F 5 "BLM41PG471SN1L" H 7400 3750 60  0001 C CNN "Part Number"
+F 6 "490-1060-1-ND" H 0   0   50  0001 C CNN "DigiKey P/N"
+F 7 "81-BLM41PG471SN1L" H 0   0   50  0001 C CNN "Mouser P/N"
 	1    7400 4150
 	1    0    0    -1
@@
 F 1 "CONN_01X02" V 8050 3950 50  0001 C CNN
 F 2 "ReflowToaster:282836-2" H 7950 3950 60  0001 C CNN
-F 3 "http://datasheet.octopart.com/282836-2-Tyco-Electronics-datasheet-11084954.pdf" H 7950 3950 60  0001 C CNN
+F 3 "http://www.te.com/commerce/DocumentDelivery/DDEController?Action=srchrtrv&DocNm=1308389_EUROSTYLE_TERMINAL_BLOCKS&DocType=CS&DocLang=English" H 7950 3950 60  0001 C CNN
 F 4 "TE Connectivity" H 7950 3950 60  0001 C CNN "Manufacturer"
 F 5 "282836-2" H 7950 3950 60  0001 C CNN "Part Number"
+F 6 "A98076-ND" H 0   0   50  0001 C CNN "DigiKey P/N"
+F 7 "571-2828362" H 0   0   50  0001 C CNN "Mouser P/N"
 	1    7950 3950
 	1    0    0    -1

Commit message: redo annotation
Parts:
- renumbered C12 to C10, C13 to C11, C10 to C7, C11 to C8, J7 to J3, U6 to U3, U5 to U4, U7 to U5, U8 to U6
Changed lines of the file:
@@
 $EndDescr
 $Comp
-L MAX31855KASA+ U7
+L MAX31855KASA+ U5
 U 1 1 540FF176
 P 5550 3950
-F 0 "U7" H 5325 4225 60  0000 L CNN
+F 0 "U5" H 5325 4225 60  0000 L CNN
 F 1 "MAX31855KASA+" H 5550 3675 60  0000 C CNN
 F 2 "SMD_Packages:SOIC-8-N" H 5550 4825 60  0001 C CNN
@@
 $EndComp
 $Comp
-L 74LVC2G34 U5
+L 74LVC2G34 U4
 U 1 1 5410697C
 P 4650 3550
-F 0 "U5" H 4550 3700 40  0000 C CNN
+F 0 "U4" H 4550 3700 40  0000 C CNN
 F 1 "74LVC2G34" H 4650 3400 40  0000 C CNN
 F 2 "SMD_Packages:SOT-23-6" H 4650 3550 60  0001 C CNN
@@
 $EndComp
 $Comp
-L 74LVC2G34 U5
+L 74LVC2G34 U4
 U 2 1 54106A65
 P 4650 3900
-F 0 "U5" H 4550 4050 40  0000 C CNN
+F 0 "U4" H 4550 4050 40  0000 C CNN
 F 1 "74LVC2G34" H 4650 3750 40  0000 C CNN
 F 2 "" H 4650 3900 60  0000 C CNN
@@
 $EndComp
 $Comp
-L +3.3V #PWR041
+L +3.3V #PWR50
 U 1 1 54106BA8
 P 4650 4300
-F 0 "#PWR041" H 4650 4260 30  0001 C CNN
+F 0 "#PWR50" H 4650 4260 30  0001 C CNN
 F 1 "+3.3V" H 4650 4410 30  0000 C CNN
 F 2 "" H 4650 4300 60  0000 C CNN
@@
 $EndComp
 $Comp
-L GND #PWR042
+L GND #PWR51
 U 1 1 54106BBC
 P 4650 4800
-F 0 "#PWR042" H 4650 4800 30  0001 C CNN
+F 0 "#PWR51" H 4650 4800 30  0001 C CNN
 F 1 "GND" H 4650 4730 30  0001 C CNN
 F 2 "" H 4650 4800 60  0000 C CNN
@@
 	4650 4300 4650 4350
 $Comp
-L C C12
+L C C10
 U 1 1 54106D7A
 P 5750 3400
-F 0 "C12" V 5700 3200 40  0000 L CNN
+F 0 "C10" V 5700 3200 40  0000 L CNN
 F 1 "0.1uF" V 5800 3450 40  0000 L CNN
 F 2 "Capacitors_SMD:c_1206" H 5788 3250 30  0001 C CNN
@@
 $EndComp
 $Comp
-L +3.3V #PWR043
+L +3.3V #PWR53
 U 1 1 54106ED2
 P 6000 3350
-F 0 "#PWR043" H 6000 3310 30  0001 C CNN
+F 0 "#PWR53" H 6000 3310 30  0001 C CNN
 F 1 "+3.3V" H 6000 3460 30  0000 C CNN
 F 2 "" H 6000 3350 60  0000 C CNN
@@
 $EndComp
 $Comp
-L GND #PWR044
+L GND #PWR52
 U 1 1 54106EE6
 P 5500 3450
-F 0 "#PWR044" H 5500 3450 30  0001 C CNN
+F 0 "#PWR52" H 5500 3450 30  0001 C CNN
 F 1 "GND" H 5500 3380 30  0001 C CNN
 F 2 "" H 5500 3450 60  0000 C CNN
@@
 Connection ~ 6000 3400
 $Comp
-L GND #PWR045
+L GND #PWR54
 U 1 1 54106BFC
 P 6000 4150
-F 0 "#PWR045" H 6000 4150 30  0001 C CNN
+F 0 "#PWR54" H 6000 4150 30  0001 C CNN
 F 1 "GND" H 6000 4080 30  0001 C CNN
 F 2 "" H 6000 4150 60  0000 C CNN
@@
 	6000 4100 6000 4150
 $Comp
-L 74LVC1T45 U6
+L 74LVC1T45 U3
 U 1 1 54106E70
 P 3750 4950
-F 0 "U6" H 3625 5250 60  0000 R CNN
+F 0 "U3" H 3625 5250 60  0000 R CNN
 F 1 "74LVC1T45" H 3775 4650 60  0000 L CNN
 F 2 "SMD_Packages:SOT-23-6" H 3750 4950 60  0001 C CNN
@@
 	5000 4950 4100 4950
 $Comp
-L C C10
+L C C7
 U 1 1 541074BF
 P 3550 4250
-F 0 "C10" H 3550 4350 40  0000 L CNN
+F 0 "C7" H 3550 4350 40  0000 L CNN
 F 1 "0.1uF" H 3556 4165 40  0000 L CNN
 F 2 "Capacitors_SMD:c_1206" H 3588 4100 30  0001 C CNN
@@
 $EndComp
 $Comp
-L C C11
+L C C8
 U 1 1 54107549
 P 3950 4250
-F 0 "C11" H 3950 4350 40  0000 L CNN
+F 0 "C8" H 3950 4350 40  0000 L CNN
 F 1 "0.1uF" H 3956 4165 40  0000 L CNN
 F 2 "Capacitors_SMD:c_1206" H 3988 4100 30  0001 C CNN
@@
 $EndComp
 $Comp
-L +3.3V #PWR046
+L +3.3V #PWR48
 U 1 1 54107680
 P 3950 4000
-F 0 "#PWR046" H 3950 3960 30  0001 C CNN
+F 0 "#PWR48" H 3950 3960 30  0001 C CNN
 F 1 "+3.3V" H 3950 4110 30  0000 C CNN
 F 2 "" H 3950 4000 60  0000 C CNN
@@
 $EndComp
 $Comp
-L +5V #PWR047
+L +5V #PWR45
 U 1 1 5410769C
 P 3550 4000
-F 0 "#PWR047" H 3550 4090 20  0001 C CNN
+F 0 "#PWR45" H 3550 4090 20  0001 C CNN
 F 1 "+5V" H 3550 4090 30  0000 C CNN
 F 2 "" H 3550 4000 60  0000 C CNN
@@
 $EndComp
 $Comp
-L GND #PWR048
+L GND #PWR49
 U 1 1 541076B0
 P 3950 4500
-F 0 "#PWR048" H 3950 4500 30  0001 C CNN
+F 0 "#PWR49" H 3950 4500 30  0001 C CNN
 F 1 "GND" H 3950 4430 30  0001 C CNN
 F 2 "" H 3950 4500 60  0000 C CNN
@@
 $EndComp
 $Comp
-L GND #PWR049
+L GND #PWR46
 U 1 1 541076C4
 P 3550 4500
-F 0 "#PWR049" H 3550 4500 30  0001 C CNN
+F 0 "#PWR46" H 3550 4500 30  0001 C CNN
 F 1 "GND" H 3550 4430 30  0001 C CNN
 F 2 "" H 3550 4500 60  0000 C CNN
@@
 	3950 4050 3950 4000
 $Comp
-L GND #PWR050
+L GND #PWR47
 U 1 1 54107794
 P 3750 5350
-F 0 "#PWR050" H 3750 5350 30  0001 C CNN
+F 0 "#PWR47" H 3750 5350 30  0001 C CNN
 F 1 "GND" H 3750 5280 30  0001 C CNN
 F 2 "" H 3750 5350 60  0000 C CNN
@@
 $EndComp
 $Comp
-L GND #PWR051
+L GND #PWR43
 U 1 1 541077B0
 P 3350 5100
-F 0 "#PWR051" H 3350 5100 30  0001 C CNN
+F 0 "#PWR43" H 3350 5100 30  0001 C CNN
 F 1 "GND" H 3350 5030 30  0001 C CNN
 F 2 "" H 3350 5100 60  0000 C CNN
@@
 	4350 3650 3200 3650
 $Comp
-L C C13
+L C C11
 U 1 1 54107DF0
 P 6450 3950
-F 0 "C13" H 6450 4050 40  0000 L CNN
+F 0 "C11" H 6450 4050 40  0000 L CNN
 F 1 "0.01uF" H 6456 3865 40  0000 L CNN
 F 2 "Capacitors_SMD:c_1206" H 6488 3800 30  0001 C CNN
@@
 	6200 4150 7150 4150
 $Comp
-L NUP2105L U8
+L NUP2105L U6
 U 1 1 541078A5
 P 6900 4450
-F 0 "U8" H 6725 4650 60  0000 R CNN
+F 0 "U6" H 6725 4650 60  0000 R CNN
 F 1 "NUP2105L" H 6925 4200 60  0000 L CNN
 F 2 "SMD_Packages:SOT-23" H 6900 4900 60  0001 C CNN
@@
 Connection ~ 6450 3750
 $Comp
-L GND #PWR052
+L GND #PWR55
 U 1 1 54107966
 P 6900 4800
-F 0 "#PWR052" H 6900 4800 30  0001 C CNN
+F 0 "#PWR55" H 6900 4800 30  0001 C CNN
 F 1 "GND" H 6900 4730 30  0001 C CNN
 F 2 "" H 6900 4800 60  0000 C CNN
@@
 Connection ~ 7000 3750
 $Comp
-L CONN_01X02 J7
+L CONN_01X02 J3
 U 1 1 5410AC42
 P 7950 3950
-F 0 "J7" H 7950 4100 50  0000 C CNN
+F 0 "J3" H 7950 4100 50  0000 C CNN
 F 1 "CONN_01X02" V 8050 3950 50  0001 C CNN
 F 2 "ReflowToaster:282836-2" H 7950 3950 60  0001 C CNN
@@
 GND
 $Comp
-L +5V #PWR053
+L +5V #PWR41
 U 1 1 5410AE90
 P 3300 2850
-F 0 "#PWR053" H 3300 2940 20  0001 C CNN
+F 0 "#PWR41" H 3300 2940 20  0001 C CNN
 F 1 "+5V" H 3300 2940 30  0000 C CNN
 F 2 "" H 3300 2850 60  0000 C CNN
@@
 $EndComp
 $Comp
-L +3.3V #PWR054
+L +3.3V #PWR44
 U 1 1 5410AEA4
 P 3400 2850
-F 0 "#PWR054" H 3400 2810 30  0001 C CNN
+F 0 "#PWR44" H 3400 2810 30  0001 C CNN
 F 1 "+3.3V" H 3400 2960 30  0000 C CNN
 F 2 "" H 3400 2850 60  0000 C CNN
@@
 $EndComp
 $Comp
-L GND #PWR055
+L GND #PWR42
 U 1 1 5410AEB8
 P 3300 3150
-F 0 "#PWR055" H 3300 3150 30  0001 C CNN
+F 0 "#PWR42" H 3300 3150 30  0001 C CNN
 F 1 "GND" H 3300 3080 30  0001 C CNN
 F 2 "" H 3300 3150 60  0000 C CNN
