File: Interface.sch (KiCad schematic (older format))
At the start: 11 parts, among them J4 CONN_02X05, Q2 PMBT3904, Q3 PMBT3904, U3 LCD8X2

Commit message: add part info for speaker
Parts:
- B1: Manufacturer (none) -> CUI; Part Number (none) -> CX-0905C
Changed lines of the file:
@@
 F 1 "SPEAKER" H 8800 1700 70  0001 C CNN
 F 2 "" H 8900 1950 60  0000 C CNN
-F 3 "" H 8900 1950 60  0000 C CNN
+F 3 " 	http://datasheet.octopart.com/CX-0905C-CUI-datasheet-40254.pdf" H 8900 1950 60  0001 C CNN
+F 4 "CUI" H 8900 1950 60  0001 C CNN "Manufacturer"
+F 5 "CX-0905C" H 8900 1950 60  0001 C CNN "Part Number"
 	1    8900 1950
 	1    0    0    -1

Commit message: last of the new footprints added; PCB started
Parts:
- B1: footprint (none) -> ReflowToaster:CX-0905C
Changed lines of the file:
@@
 F 0 "B1" H 8800 2200 70  0000 C CNN
 F 1 "SPEAKER" H 8800 1700 70  0001 C CNN
-F 2 "" H 8900 1950 60  0000 C CNN
-F 3 " 	http://datasheet.octopart.com/CX-0905C-CUI-datasheet-40254.pdf" H 8900 1950 60  0001 C CNN
+F 2 "ReflowToaster:CX-0905C" H 8900 1950 60  0001 C CNN
+F 3 "http://datasheet.octopart.com/CX-0905C-CUI-datasheet-40254.pdf" H 8900 1950 60  0001 C CNN
 F 4 "CUI" H 8900 1950 60  0001 C CNN "Manufacturer"
 F 5 "CX-0905C" H 8900 1950 60  0001 C CNN "Part Number"

Commit message: components tagged with vendor part IDs
Parts:
- B1: DigiKey P/N (none) -> 102-1285-ND; Mouser P/N (none) -> 254-EMB105-RO; Note (none) -> sub Kobitone 254-EMB105-RO when ordering from Mouser
- J4: DigiKey P/N (none) -> 952-2380-ND; Manufacturer (none) -> Harwin; Mouser P/N (none) -> 855-M20-9980545; Part Number (none) -> M20-9980545
- Q2, Q3: DigiKey P/N (none) -> 568-1741-1-ND; Mouser P/N (none) -> 771-PMBT3904-T/R
- R10, R7, R9: DigiKey P/N (none) -> P10KECT-ND; Manufacturer (none) -> Panasonic; Mouser P/N (none) -> 667-ERJ-8GEYJ103V; Part Number (none) -> ERJ-8GEYJ103V
- R5: DigiKey P/N (none) -> P1KECT-ND; Manufacturer (none) -> Panasonic; Mouser P/N (none) -> 667-ERJ-8GEYJ102V; Part Number (none) -> ERJ-8GEYJ102V
- R6: DigiKey P/N (none) -> 3319P-103-ND; Mouser P/N (none) -> 652-3319P-1-103
- R8: DigiKey P/N (none) -> P47KECT-ND; Manufacturer (none) -> Panasonic; Mouser P/N (none) -> 667-ERJ-8GEYJ473V; Part Number (none) -> ERJ-8GEYJ473V
- U3: DigiKey P/N (none) -> NHD-0208AZ-FL-YBW-ND; Mouser P/N (none) -> 763-0208AZ-FL-YBW
Changed lines of the file:
@@
 F 1 "CONN_02X05" H 5000 3350 50  0001 C CNN
 F 2 "Pin_Headers:Pin_Header_Straight_2x05" H 5000 2450 60  0001 C CNN
-F 3 "" H 5000 2450 60  0000 C CNN
+F 3 "http://harwin.com/includes/pdfs/60page147.pdf" H 8900 1950 60  0001 C CNN
+F 4 "Harwin" H 8900 1950 60  0001 C CNN "Manufacturer"
+F 5 "M20-9980545" H 8900 1950 60  0001 C CNN "Part Number"
+F 6 "952-2380-ND" H 0   0   50  0001 C CNN "DigiKey P/N"
+F 7 "855-M20-9980545" H 0   0   50  0001 C CNN "Mouser P/N"
 	1    5000 3650
 	1    0    0    -1
@@
 F 1 "1k" V 5182 2361 40  0000 L CNN
 F 2 "Capacitors_SMD:c_1206" H 5080 2250 30  0001 C CNN
-F 3 "" H 5175 2360 30  0000 C CNN
+F 3 "http://industrial.panasonic.com/www-cgi/jvcr13pz.cgi?E+PZ+3+AOA0001+ERJ8GEYJ102V+7+WW" H 7125 5260 30  0001 C CNN
+F 4 "Panasonic" H 3500 3550 60  0001 C CNN "Manufacturer"
+F 5 "ERJ-8GEYJ102V" H 3500 3550 60  0001 C CNN "Part Number"
+F 6 "P1KECT-ND" H 0   0   50  0001 C CNN "DigiKey P/N"
+F 7 "667-ERJ-8GEYJ102V" H 0   0   50  0001 C CNN "Mouser P/N"
 	1    5150 2250
 	0    1    1    0
@@
 F 1 "47k" V 8082 5811 40  0000 L CNN
 F 2 "Capacitors_SMD:c_1206" V 7980 5700 30  0001 C CNN
-F 3 "" H 8075 5810 30  0000 C CNN
+F 3 "http://industrial.panasonic.com/www-cgi/jvcr13pz.cgi?E+PZ+3+AOA0001+ERJ8GEYJ473V+7+WW" H 7125 5260 30  0001 C CNN
+F 4 "Panasonic" H 3500 3550 60  0001 C CNN "Manufacturer"
+F 5 "ERJ-8GEYJ473V" H 3500 3550 60  0001 C CNN "Part Number"
+F 6 "P47KECT-ND" H 0   0   50  0001 C CNN "DigiKey P/N"
+F 7 "667-ERJ-8GEYJ473V" H 0   0   50  0001 C CNN "Mouser P/N"
 	1    8050 5700
 	0    1    1    0
@@
 F 1 "PMBT3904" H 8550 5550 50  0000 R CNN
 F 2 "SMD_Packages:SOT-23" H 8550 6650 60  0001 C CNN
-F 3 "http://datasheet.octopart.com/PMBT3904-Philips-datasheet-90020.pdf" H 8550 6750 60  0001 C CNN
-F 4 "NXP" H 8550 6825 60  0001 C CNN "Manufacturer"
-F 5 "PMBT3904" H 8550 6900 60  0001 C CNN "Part Number"
+F 3 "http://www.nxp.com/documents/data_sheet/PMBT3904.pdf" H 8500 3350 60  0001 C CNN
+F 4 "NXP" H 8500 3425 60  0001 C CNN "Manufacturer"
+F 5 "PMBT3904" H 8500 3500 60  0001 C CNN "Part Number"
+F 6 "568-1741-1-ND" H 0   0   50  0001 C CNN "DigiKey P/N"
+F 7 "771-PMBT3904-T/R" H 0   0   50  0001 C CNN "Mouser P/N"
 	1    8550 5700
 	1    0    0    -1
@@
 F 1 "10k" V 8032 2411 40  0000 L CNN
 F 2 "Capacitors_SMD:c_1206" V 7930 2300 30  0001 C CNN
-F 3 "" H 8025 2410 30  0000 C CNN
+F 3 "http://industrial.panasonic.com/www-cgi/jvcr13pz.cgi?E+PZ+3+AOA0001+ERJ8GEYJ103V+7+WW" H 7125 5260 30  0001 C CNN
+F 4 "Panasonic" H 3500 3550 60  0001 C CNN "Manufacturer"
+F 5 "ERJ-8GEYJ103V" H 3500 3550 60  0001 C CNN "Part Number"
+F 6 "P10KECT-ND" H 0   0   50  0001 C CNN "DigiKey P/N"
+F 7 "667-ERJ-8GEYJ103V" H 0   0   50  0001 C CNN "Mouser P/N"
 	1    8000 2300
 	0    1    1    0
@@
 F 1 "PMBT3904" H 8500 2150 50  0000 R CNN
 F 2 "SMD_Packages:SOT-23" H 8500 3250 60  0001 C CNN
-F 3 "http://datasheet.octopart.com/PMBT3904-Philips-datasheet-90020.pdf" H 8500 3350 60  0001 C CNN
+F 3 "http://www.nxp.com/documents/data_sheet/PMBT3904.pdf" H 8500 3350 60  0001 C CNN
 F 4 "NXP" H 8500 3425 60  0001 C CNN "Manufacturer"
 F 5 "PMBT3904" H 8500 3500 60  0001 C CNN "Part Number"
+F 6 "568-1741-1-ND" H 0   0   50  0001 C CNN "DigiKey P/N"
+F 7 "771-PMBT3904-T/R" H 0   0   50  0001 C CNN "Mouser P/N"
 	1    8500 2300
 	1    0    0    -1
@@
 F 1 "SPEAKER" H 8800 1700 70  0001 C CNN
 F 2 "ReflowToaster:CX-0905C" H 8900 1950 60  0001 C CNN
-F 3 "http://datasheet.octopart.com/CX-0905C-CUI-datasheet-40254.pdf" H 8900 1950 60  0001 C CNN
+F 3 "http://www.cui.com/product/resource/digikeypdf/cx-0905c.pdf" H 8900 1950 60  0001 C CNN
 F 4 "CUI" H 8900 1950 60  0001 C CNN "Manufacturer"
 F 5 "CX-0905C" H 8900 1950 60  0001 C CNN "Part Number"
+F 6 "102-1285-ND" H 0   0   50  0001 C CNN "DigiKey P/N"
+F 7 "254-EMB105-RO" H 0   0   50  0001 C CNN "Mouser P/N"
+F 8 "sub Kobitone 254-EMB105-RO when ordering from Mouser" H 0 0 50 0001 C CNN "Note"
 	1    8900 1950
 	1    0    0    -1
@@
 F 4 "Newhaven Display" H 8300 3800 60  0001 C CNN "Manufacturer"
 F 5 "NHD-0208AZ-FL-YBW" H 8300 3800 60  0001 C CNN "Part Number"
+F 6 "NHD-0208AZ-FL-YBW-ND" H 0   0   50  0001 C CNN "DigiKey P/N"
+F 7 "763-0208AZ-FL-YBW" H 0   0   50  0001 C CNN "Mouser P/N"
 	1    8300 3800
 	1    0    0    -1
@@
 F 1 "10k" V 7782 4861 40  0000 L CNN
 F 2 "ReflowToaster:3319P-1-103" V 7680 4750 30  0001 C CNN
-F 3 "http://datasheet.octopart.com/3319P-1-103-Bourns-datasheet-4388.pdf" H 7775 4860 30  0001 C CNN
+F 3 "http://www.bourns.com/data/global/pdfs/3319.pdf" H 7775 4860 30  0001 C CNN
 F 4 "Bourns" V 7750 4750 60  0001 C CNN "Manufacturer"
 F 5 "3319P-1-103" V 7750 4750 60  0001 C CNN "Part Number"
+F 6 "3319P-103-ND" H 0   0   50  0001 C CNN "DigiKey P/N"
+F 7 "652-3319P-1-103" H 0   0   50  0001 C CNN "Mouser P/N"
 	1    7750 4750
 	0    1    1    0
@@
 F 1 "10k" V 2682 3561 40  0000 L CNN
 F 2 "Capacitors_SMD:c_1206" V 2580 3450 30  0001 C CNN
-F 3 "" H 2675 3560 30  0000 C CNN
+F 3 "http://industrial.panasonic.com/www-cgi/jvcr13pz.cgi?E+PZ+3+AOA0001+ERJ8GEYJ103V+7+WW" H 7125 5260 30  0001 C CNN
+F 4 "Panasonic" H 3500 3550 60  0001 C CNN "Manufacturer"
+F 5 "ERJ-8GEYJ103V" H 3500 3550 60  0001 C CNN "Part Number"
+F 6 "P10KECT-ND" H 0   0   50  0001 C CNN "DigiKey P/N"
+F 7 "667-ERJ-8GEYJ103V" H 0   0   50  0001 C CNN "Mouser P/N"
 	1    2650 3450
 	1    0    0    -1
@@
 F 1 "10k" V 2682 4211 40  0000 L CNN
 F 2 "Capacitors_SMD:c_1206" V 2580 4100 30  0001 C CNN
-F 3 "" H 2675 4210 30  0000 C CNN
+F 3 "http://industrial.panasonic.com/www-cgi/jvcr13pz.cgi?E+PZ+3+AOA0001+ERJ8GEYJ103V+7+WW" H 7125 5260 30  0001 C CNN
+F 4 "Panasonic" H 3500 3550 60  0001 C CNN "Manufacturer"
+F 5 "ERJ-8GEYJ103V" H 3500 3550 60  0001 C CNN "Part Number"
+F 6 "P10KECT-ND" H 0   0   50  0001 C CNN "DigiKey P/N"
+F 7 "667-ERJ-8GEYJ103V" H 0   0   50  0001 C CNN "Mouser P/N"
 	1    2650 4100
 	1    0    0    -1

Commit message: fix incorrect vendor part number
Parts:
- R5: DigiKey P/N P1KECT-ND -> P1.0KECT-ND
Changed lines of the file:
@@
 F 4 "Panasonic" H 3500 3550 60  0001 C CNN "Manufacturer"
 F 5 "ERJ-8GEYJ102V" H 3500 3550 60  0001 C CNN "Part Number"
-F 6 "P1KECT-ND" H 0   0   50  0001 C CNN "DigiKey P/N"
+F 6 "P1.0KECT-ND" H 0   0   50  0001 C CNN "DigiKey P/N"
 F 7 "667-ERJ-8GEYJ102V" H 0   0   50  0001 C CNN "Mouser P/N"
 	1    5150 2250
@@
 F 6 "102-1285-ND" H 0   0   50  0001 C CNN "DigiKey P/N"
 F 7 "254-EMB105-RO" H 0   0   50  0001 C CNN "Mouser P/N"
-F 8 "sub Kobitone 254-EMB105-RO when ordering from Mouser" H 0 0 50 0001 C CNN "Note"
+F 8 "sub Kobitone 254-EMB105-RO when ordering from Mouser" H 0   0   50  0001 C CNN "Note"
 	1    8900 1950
 	1    0    0    -1

Commit message: redo annotation
Parts:
- renumbered R8 to R10, R9 to R5, R10 to R6, R5 to R7, R6 to R8, R7 to R9, U3 to U7
Changed lines of the file:
@@
 $EndComp
 $Comp
-L GND #PWR056
+L GND #PWR58
 U 1 1 54114BA9
 P 4700 3900
-F 0 "#PWR056" H 4700 3900 30  0001 C CNN
+F 0 "#PWR58" H 4700 3900 30  0001 C CNN
 F 1 "GND" H 4700 3830 30  0001 C CNN
 F 2 "" H 4700 3900 60  0000 C CNN
@@
 $EndComp
 $Comp
-L +5V #PWR057
+L +5V #PWR57
 U 1 1 54114BCF
 P 4700 3400
-F 0 "#PWR057" H 4700 3490 20  0001 C CNN
+F 0 "#PWR57" H 4700 3490 20  0001 C CNN
 F 1 "+5V" H 4700 3490 30  0000 C CNN
 F 2 "" H 4700 3400 60  0000 C CNN
@@
 GND
 $Comp
-L +5V #PWR058
+L +5V #PWR59
 U 1 1 54114D7A
 P 5300 5300
-F 0 "#PWR058" H 5300 5390 20  0001 C CNN
+F 0 "#PWR59" H 5300 5390 20  0001 C CNN
 F 1 "+5V" H 5300 5390 30  0000 C CNN
 F 2 "" H 5300 5300 60  0000 C CNN
@@
 $EndComp
 $Comp
-L GND #PWR059
+L GND #PWR60
 U 1 1 54114D8F
 P 5300 5550
-F 0 "#PWR059" H 5300 5550 30  0001 C CNN
+F 0 "#PWR60" H 5300 5550 30  0001 C CNN
 F 1 "GND" H 5300 5480 30  0001 C CNN
 F 2 "" H 5300 5550 60  0000 C CNN
@@
 D4
 $Comp
-L R R5
+L R R7
 U 1 1 54114DE5
 P 5150 2250
-F 0 "R5" V 5115 2155 40  0000 R CNN
+F 0 "R7" V 5115 2155 40  0000 R CNN
 F 1 "1k" V 5182 2361 40  0000 L CNN
 F 2 "Capacitors_SMD:c_1206" H 5080 2250 30  0001 C CNN
@@
 D5
 $Comp
-L R R8
+L R R10
 U 1 1 54115058
 P 8050 5700
-F 0 "R8" V 8015 5605 40  0000 R CNN
+F 0 "R10" V 8015 5605 40  0000 R CNN
 F 1 "47k" V 8082 5811 40  0000 L CNN
 F 2 "Capacitors_SMD:c_1206" V 7980 5700 30  0001 C CNN
@@
 SSR
 $Comp
-L GND #PWR060
+L GND #PWR68
 U 1 1 5411514F
 P 8650 5950
-F 0 "#PWR060" H 8650 5950 30  0001 C CNN
+F 0 "#PWR68" H 8650 5950 30  0001 C CNN
 F 1 "GND" H 8650 5880 30  0001 C CNN
 F 2 "" H 8650 5950 60  0000 C CNN
@@
 D6
 $Comp
-L R R7
+L R R9
 U 1 1 5411526E
 P 8000 2300
-F 0 "R7" V 7965 2205 40  0000 R CNN
+F 0 "R9" V 7965 2205 40  0000 R CNN
 F 1 "10k" V 8032 2411 40  0000 L CNN
 F 2 "Capacitors_SMD:c_1206" V 7930 2300 30  0001 C CNN
@@
 $EndComp
 $Comp
-L GND #PWR061
+L GND #PWR67
 U 1 1 54115390
 P 8600 2550
-F 0 "#PWR061" H 8600 2550 30  0001 C CNN
+F 0 "#PWR67" H 8600 2550 30  0001 C CNN
 F 1 "GND" H 8600 2480 30  0001 C CNN
 F 2 "" H 8600 2550 60  0000 C CNN
@@
 $EndComp
 $Comp
-L +5V #PWR062
+L +5V #PWR66
 U 1 1 5411574F
 P 8600 1800
-F 0 "#PWR062" H 8600 1890 20  0001 C CNN
+F 0 "#PWR66" H 8600 1890 20  0001 C CNN
 F 1 "+5V" H 8600 1890 30  0000 C CNN
 F 2 "" H 8600 1800 60  0000 C CNN
@@
 $EndComp
 $Comp
-L LCD8X2 U3
+L LCD8X2 U7
 U 1 1 54111EAD
 P 8300 3800
-F 0 "U3" H 7500 4200 40  0000 C CNN
+F 0 "U7" H 7500 4200 40  0000 C CNN
 F 1 "LCD8X2" H 9000 4200 40  0000 C CNN
 F 2 "ReflowToaster:LCD_8x2" H 8300 3750 35  0000 C CIN
@@
 $EndComp
 $Comp
-L GND #PWR063
+L GND #PWR62
 U 1 1 54111FC8
 P 7550 4350
-F 0 "#PWR063" H 7550 4350 30  0001 C CNN
+F 0 "#PWR62" H 7550 4350 30  0001 C CNN
 F 1 "GND" H 7550 4280 30  0001 C CNN
 F 2 "" H 7550 4350 60  0000 C CNN
@@
 $EndComp
 $Comp
-L +5V #PWR064
+L +5V #PWR63
 U 1 1 541120A4
 P 7650 4350
-F 0 "#PWR064" H 7650 4440 20  0001 C CNN
+F 0 "#PWR63" H 7650 4440 20  0001 C CNN
 F 1 "+5V" H 7650 4440 30  0000 C CNN
 F 2 "" H 7650 4350 60  0000 C CNN
@@
 $EndComp
 $Comp
-L GND #PWR065
+L GND #PWR70
 U 1 1 54112123
 P 9050 4350
-F 0 "#PWR065" H 9050 4350 30  0001 C CNN
+F 0 "#PWR70" H 9050 4350 30  0001 C CNN
 F 1 "GND" H 9050 4280 30  0001 C CNN
 F 2 "" H 9050 4350 60  0000 C CNN
@@
 $EndComp
 $Comp
-L +5V #PWR066
+L +5V #PWR69
 U 1 1 5411213F
 P 8950 4350
-F 0 "#PWR066" H 8950 4440 20  0001 C CNN
+F 0 "#PWR69" H 8950 4440 20  0001 C CNN
 F 1 "+5V" H 8950 4440 30  0000 C CNN
 F 2 "" H 8950 4350 60  0000 C CNN
@@
 $EndComp
 $Comp
-L POT R6
+L POT R8
 U 1 1 5411310D
 P 7750 4750
-F 0 "R6" V 7715 4655 40  0000 R CNN
+F 0 "R8" V 7715 4655 40  0000 R CNN
 F 1 "10k" V 7782 4861 40  0000 L CNN
 F 2 "ReflowToaster:3319P-1-103" V 7680 4750 30  0001 C CNN
@@
 	7750 4300 7750 4550
 $Comp
-L GND #PWR067
+L GND #PWR64
 U 1 1 54113876
 P 7950 4350
-F 0 "#PWR067" H 7950 4350 30  0001 C CNN
+F 0 "#PWR64" H 7950 4350 30  0001 C CNN
 F 1 "GND" H 7950 4280 30  0001 C CNN
 F 2 "" H 7950 4350 60  0000 C CNN
@@
 	7950 4350 7950 4300
 $Comp
-L GND #PWR068
+L GND #PWR61
 U 1 1 541138CC
 P 7450 4800
-F 0 "#PWR068" H 7450 4800 30  0001 C CNN
+F 0 "#PWR61" H 7450 4800 30  0001 C CNN
 F 1 "GND" H 7450 4730 30  0001 C CNN
 F 2 "" H 7450 4800 60  0000 C CNN
@@
 $EndComp
 $Comp
-L +5V #PWR069
+L +5V #PWR65
 U 1 1 541138E9
 P 8050 4700
-F 0 "#PWR069" H 8050 4790 20  0001 C CNN
+F 0 "#PWR65" H 8050 4790 20  0001 C CNN
 F 1 "+5V" H 8050 4790 30  0000 C CNN
 F 2 "" H 8050 4700 60  0000 C CNN
@@
 	8850 4300 8850 4350
 $Comp
-L R R9
+L R R5
 U 1 1 54114022
 P 2650 3450
-F 0 "R9" V 2615 3355 40  0000 R CNN
+F 0 "R5" V 2615 3355 40  0000 R CNN
 F 1 "10k" V 2682 3561 40  0000 L CNN
 F 2 "Capacitors_SMD:c_1206" V 2580 3450 30  0001 C CNN
@@
 $EndComp
 $Comp
-L R R10
+L R R6
 U 1 1 541140C9
 P 2650 4100
-F 0 "R10" V 2615 4005 40  0000 R CNN
+F 0 "R6" V 2615 4005 40  0000 R CNN
 F 1 "10k" V 2682 4211 40  0000 L CNN
 F 2 "Capacitors_SMD:c_1206" V 2580 4100 30  0001 C CNN
@@
 Connection ~ 2650 3750
 $Comp
-L +5V #PWR070
+L +5V #PWR56
 U 1 1 541142D7
 P 2650 3150
-F 0 "#PWR070" H 2650 3240 20  0001 C CNN
+F 0 "#PWR56" H 2650 3240 20  0001 C CNN
 F 1 "+5V" H 2650 3240 30  0000 C CNN
 F 2 "" H 2650 3150 60  0000 C CNN

Commit message: more work
Parts:
- added J5, J6: CONN_02X08, symbol CONN_02X08
Other:
- note added: "Do Not Place"
Changed lines of the file:
@@
 	2700 3800 2650 3800
 Connection ~ 2650 3800
+$Comp
+L CONN_02X08 J5
+U 1 1 5413BC75
+P 1500 1550
+F 0 "J5" H 1500 2000 50  0000 C CNN
+F 1 "CONN_02X08" V 1500 1550 50  0000 C CNN
+F 2 "" H 1500 350 60  0000 C CNN
+F 3 "http://www.sullinscorp.com/drawings/78_P(N)PxCxxxLFBN-RC,_10492-G.pdf" H 1500 350 60  0001 C CNN
+F 4 "Sullins" H 1500 1550 60  0001 C CNN "Manufacturer"
+F 5 "PPTC082LFBN-RC" H 1500 1550 60  0001 C CNN "Part Number"
+F 6 "S7076-ND" H 1500 1550 60  0001 C CNN "DigiKey P/N"
+F 7 "649-76342-408LF" H 1500 1550 60  0001 C CNN "Mouser P/N"
+F 8 "Do Not Place - part included for BOM generation; sub FCI 76342-408LF when ordering from Mouser" H 1500 1550 60  0001 C CNN "Note"
+	1    1500 1550
+	1    0    0    -1
+$EndComp
+$Comp
+L CONN_02X08 J6
+U 1 1 5413BD18
+P 2100 1550
+F 0 "J6" H 2100 2000 50  0000 C CNN
+F 1 "CONN_02X08" V 2100 1550 50  0000 C CNN
+F 2 "" H 2100 350 60  0000 C CNN
+F 3 "http://harwin.com/includes/pdfs/M20-976.pdf" H 2100 350 60  0001 C CNN
+F 4 "Harwin" H 2100 1550 60  0001 C CNN "Manufacturer"
+F 5 "M20-9760842" H 2100 1550 60  0001 C CNN "Part Number"
+F 6 "952-1817-ND" H 2100 1550 60  0001 C CNN "DigiKey P/N"
+F 7 "855-M20-9760842" H 2100 1550 60  0001 C CNN "Mouser P/N"
+F 8 "Do Not Place - part included for BOM generation" H 2100 1550 60  0001 C CNN "Note"
+	1    2100 1550
+	1    0    0    -1
+$EndComp
+Wire Notes Line
+	850  700  2700 700
+Wire Notes Line
+	2700 700  2700 2050
+Wire Notes Line
+	2700 2050 850  2050
+Wire Notes Line
+	850  2050 850  700
+Text Notes 1300 950  0    100  ~ 0
+Do Not Place
 $EndSCHEMATC
