File: ReflowToaster.kicad_pcb (KiCad board)
At the start: 2 copper layers, 50 x 70 mm, 44 parts, among them J2 USB-Micro-B, J3 USB-Micro-B, J4 CONN_02X05, J7 CONN_01X02, P1 CONN_02X03, Q1 FDN340P, Q2 PMBT3904, Q3 PMBT3904, U1 ATMEGA32U4-A, U2 MCP1700T-3302E/TT, U3 LCD8X2, U5 74LVC2G34, U6 74LVC1T45, U7 MAX31855KASA+, U8 NUP2105L, X1 16MHz

Commit message: more work
Parts:
- removed C12: 0.1uF, Capacitors_SMD:c_1206
- removed C13: 0.01uF, Capacitors_SMD:c_1206
- removed J7: CONN_01X02, ReflowToaster:282836-2
- removed U8: NUP2105L, SMD_Packages:SOT-23
- added C7: 0.1uF, Capacitors_SMD:c_1206, F.Cu at (74.3, 191.0)
- added C8: 0.1uF, Capacitors_SMD:c_1206, F.Cu at (87.8, 179.9)
- added J1: USB-Micro-B, ReflowToaster:FCI_10118192-0001LF, F.Cu at (102.0, 180.0)
- added MH: MountingHole_2mm, ReflowToaster:MountingHole_2mm, F.Cu at (134.3, 130.4)
- added U4: 74LVC2G34, SMD_Packages:SOT-23-6, F.Cu at (87.6, 175.8)
- B1, J4: moved to F.Cu
- C11: value 0.1uF -> 0.01uF
- C2, C3: value 0.1uF -> 1uF
- C5, C6: value 1uF -> 0.1uF
- J3: value USB-Micro-B -> CONN_01X02; footprint ReflowToaster:FCI_10118192-0001LF -> ReflowToaster:282836-2
- R10: value 10k -> 47k
- R5: value 1k -> 10k
- R6: footprint ReflowToaster:3319P-1-103 -> Capacitors_SMD:c_1206; moved to F.Cu
- R7: value 10k -> 1k
- R8: value 47k -> 10k; footprint Capacitors_SMD:c_1206 -> ReflowToaster:3319P-1-103
- U1: value ATMEGA32U4-A -> MCP1700T-3302E/TT; footprint SMD_Packages:TQFP-44 -> SMD_Packages:SOT-23
- U2: value MCP1700T-3302E/TT -> ATMEGA32U4-A; footprint SMD_Packages:SOT-23 -> SMD_Packages:TQFP-44
- U3: value LCD8X2 -> 74LVC1T45; footprint ReflowToaster:LCD_8x2 -> SMD_Packages:SOT-23-6
- U5: value 74LVC2G34 -> MAX31855KASA+; footprint SMD_Packages:SOT-23-6 -> SMD_Packages:SOIC-8-N
- U6: value 74LVC1T45 -> NUP2105L; footprint SMD_Packages:SOT-23-6 -> SMD_Packages:SOT-23
- U7: value MAX31855KASA+ -> LCD8X2; footprint SMD_Packages:SOIC-8-N -> ReflowToaster:LCD_8x2
- moved L1 191.6 mm to (18.4, 192.5)
- moved C6 191.3 mm to (27.7, 192.5)
- moved Q3 182.9 mm to (18.7, 168.6)
- moved R10 179.7 mm to (28.9, 168.8)
- moved B1 177.9 mm to (82.5, 159.2)
- moved C2 176.4 mm to (40.6, 188.0)
- moved C4 171.9 mm to (37.5, 192.5)
- moved U3 171.2 mm to (74.1, 186.9)
- moved R6 165.7 mm to (24.0, 168.8), turned to 0 degrees
- moved U1 165.6 mm to (20.8, 189.1)
- moved C3 161.1 mm to (32.6, 192.5)
- moved X1 159.5 mm to (34.0, 186.2)
- moved R7 157.2 mm to (38.7, 168.8)
- moved VR2 155.2 mm to (21.7, 192.0)
- moved R4 152.1 mm to (50.4, 185.9)
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Connections:
- C1 pad 1: Net-(C1-Pad1) -> +5V
- C10 pad 1: +5V -> +3.3V
- C11 pad 1: +3.3V -> Net-(C11-Pad1)
- C11 pad 2: GND -> Net-(C11-Pad2)
- C2 pad 1: +5V -> +3.3V
- C3 pad 1: /DuinoModSingle/AREF -> Net-(C3-Pad1)
- C4 pad 1: Net-(C4-Pad1) -> /DuinoModSingle/AREF
- C5 pad 1: +3.3V -> +5V
- C6 pad 1: +5V -> Net-(C6-Pad1)
- L1 pad 2: Net-(C4-Pad1) -> Net-(C6-Pad1)
- L2 pad 1: Net-(C13-Pad1) -> Net-(C11-Pad1)
- L2 pad 2: Net-(J7-Pad1) -> Net-(J3-Pad1)
- L3 pad 1: Net-(C13-Pad2) -> Net-(C11-Pad2)
- L3 pad 2: Net-(J7-Pad2) -> Net-(J3-Pad2)
- Q1 pad G: Net-(J3-Pad1) -> Net-(J1-Pad1)
- R10 pad 1: BTN1 -> Net-(Q3-Pad1)
- R10 pad 2: BTN2 -> /DuinoModSingle/5/PWM
- R3 pad 1: +5V -> GND
- R3 pad 2: /DuinoModSingle/~RESET -> Net-(R3-Pad2)
- R4 pad 1: GND -> +5V
- R4 pad 2: Net-(R4-Pad2) -> /DuinoModSingle/~RESET
- R5 pad 1: LED -> +5V
- R5 pad 2: /DuinoModSingle/4/A6 -> BTN1
- R6 pad 1: +5V -> BTN1
- R6 pad 2: GND -> BTN2
- R7 pad 1: Net-(Q2-Pad1) -> LED
- R7 pad 2: /DuinoModSingle/6/PWM/A8 -> /DuinoModSingle/4/A6
- R8 pad 1: Net-(Q3-Pad1) -> +5V
- R8 pad 2: /DuinoModSingle/5/PWM -> GND
- R9 pad 1: +5V -> Net-(Q2-Pad1)
- R9 pad 2: BTN1 -> /DuinoModSingle/6/PWM/A8
- U1 pad 1: /DuinoModSingle/7 -> GND
- U1 pad 2: +5V -> +3.3V
- U1 pad 3: Net-(R1-Pad1) -> +5V
- U2 pad 1: GND -> /DuinoModSingle/7
- U2 pad 2: +3.3V -> +5V
- U2 pad 3: +5V -> Net-(R1-Pad1)
- U3 pad 1: GND -> +5V
- U3 pad 2: +5V -> GND
- U3 pad 3: Net-(R6-Pad3) -> /DuinoModSingle/A3
- U3 pad 4: /DuinoModSingle/7 -> Net-(U3-Pad4)
- U3 pad 6: /DuinoModSingle/8/A9 -> +3.3V
- U5 pad 1: /DuinoModSingle/A1 -> GND
- U5 pad 2: GND -> Net-(C11-Pad2)
- U5 pad 3: /DuinoModSingle/A2 -> Net-(C11-Pad1)
- U5 pad 4: Net-(U5-Pad4) -> +3.3V
- U5 pad 5: VCC -> Net-(U4-Pad6)
- U5 pad 6: Net-(U5-Pad6) -> Net-(U4-Pad4)
- U6 pad 1: +5V -> Net-(C11-Pad2)
- U6 pad 2: GND -> Net-(C11-Pad1)
- U6 pad 3: /DuinoModSingle/A3 -> GND
- U7 pad 2: Net-(C13-Pad2) -> +5V
- U7 pad 3: Net-(C13-Pad1) -> Net-(R8-Pad3)
- U7 pad 4: +3.3V -> /DuinoModSingle/7
- U7 pad 5: Net-(U5-Pad6) -> GND
- U7 pad 6: Net-(U5-Pad4) -> /DuinoModSingle/8/A9
- U7 pad 7: Net-(U6-Pad4) -> Net-(U7-Pad7)
- X1 pad 1: Net-(U1-Pad17) -> Net-(U2-Pad17)
- X1 pad 2: Net-(U1-Pad16) -> Net-(U2-Pad16)
Other:
- board size 50 x 70 mm -> 50 x 63.5 mm
